Commit message: able to load, modify and save new urdf. still trying to figure out how to scale human part

File: assistive_gym/envs/assets/human/human_pip.urdf (robot description, URDF)
Before this commit: robot human, 95 links, 94 joints
Links:
- link left_elbow_limb: geometry collision capsule length=0.2 radius=0.023
- link left_hip_rx: mass 1e-05 -> 0
- link left_hip_ry: mass 1e-05 -> 0; geometry collision sphere radius=0.000000
- link left_hip_rz: mass 1e-05 -> 0; geometry collision sphere radius=0
- link left_lowarm_limb: geometry collision capsule length=0.2 radius=0.023
- link right_elbow_limb: geometry collision capsule length=0.2 radius=0.023
- link right_lowarm_limb: geometry collision capsule length=0.2 radius=0.023
