Commit message: more realistic human urdf. play with human mesh

File: assistive_gym/envs/assets/human/human_pip_original.urdf (robot description, URDF)
Before this commit: robot human, 95 links, 94 joints
Links:
- link head_limb: geometry collision sphere radius=0.07
- link left_elbow_limb: geometry collision capsule length=0.2 radius=0.023
- link left_knee_limb: geometry collision capsule length=0.29605029420748488 radius=0.05
- link left_shoulder_limb: geometry collision sphere radius=0.05
- link neck_limb: geometry collision sphere radius=0.07
- link right_elbow_limb: geometry collision capsule length=0.2 radius=0.023
- link right_knee_limb: geometry collision capsule length=0.29416381919362977 radius=0.05
- link right_shoulder_limb: geometry collision sphere radius=0.05
- link root: geometry collision sphere radius=0.07
- link spine_2_limb: geometry collision sphere radius=0.05
- link spine_3_limb: geometry collision sphere radius=0.05
- link spine_4_limb: geometry collision sphere radius=0.05
