Commit message: generate geom under custom folder

File: assistive_gym/envs/assets/human/ref_mesh.urdf (robot description, URDF)
Before this commit: robot human, 94 links, 93 joints
Links:
- link head_limb: geometry collision mesh filename=./meshes/Head.obj scale=1.00000 1.00000 1.00000; visual mesh filename=./meshes/Head.obj scale=1.00000 1.00000 1.00000
- link left_ankle_limb: geometry collision mesh filename=./meshes/L_Ankle.obj scale=1.00000 1.00000 1.00000; visual mesh filename=./meshes/L_Ankle.obj scale=1.00000 1.00000 1.00000
- link left_clavicle_limb: geometry collision mesh filename=./meshes/L_Collar.obj scale=1.00000 1.00000 1.00000; visual mesh filename=./meshes/L_Collar.obj scale=1.00000 1.00000 1.00000
- link left_elbow_limb: geometry collision mesh filename=./meshes/L_Elbow.obj scale=1.00000 1.00000 1.00000; visual mesh filename=./meshes/L_Elbow.obj scale=1.00000 1.00000 1.00000
- link left_foot_limb: geometry collision mesh filename=./meshes/L_Foot.obj scale=1.00000 1.00000 1.00000; visual mesh filename=./meshes/L_Foot.obj scale=1.00000 1.00000 1.00000
- link left_hand_limb: geometry collision mesh filename=./meshes/L_Hand.obj scale=1.00000 1.00000 1.00000; visual mesh filename=./meshes/L_Hand.obj scale=1.00000 1.00000 1.00000
- link left_hip_limb: geometry collision mesh filename=./meshes/L_Hip.obj scale=1.00000 1.00000 1.00000; visual mesh filename=./meshes/L_Hip.obj scale=1.00000 1.00000 1.00000
- link left_knee_limb: geometry collision mesh filename=./meshes/L_Knee.obj scale=1.00000 1.00000 1.00000; visual mesh filename=./meshes/L_Knee.obj scale=1.00000 1.00000 1.00000
- link left_lowarm_limb: geometry collision mesh filename=./meshes/L_Wrist.obj scale=1.00000 1.00000 1.00000; visual mesh filename=./meshes/L_Wrist.obj scale=1.00000 1.00000 1.00000
- link left_shoulder_limb: geometry collision mesh filename=./meshes/L_Shoulder.obj scale=1.00000 1.00000 1.00000; visual mesh filename=./meshes/L_Shoulder.obj scale=1.00000 1.00000 1.00000
- link neck_limb: geometry collision mesh filename=./meshes/Neck.obj scale=1.00000 1.00000 1.00000; visual mesh filename=./meshes/Neck.obj scale=1.00000 1.00000 1.00000
- link pelvis_limb: geometry collision mesh filename=./meshes/Pelvis.obj scale=1.00000 1.00000 1.00000; visual mesh filename=./meshes/Pelvis.obj scale=1.00000 1.00000 1.00000
- link right_ankle_limb: geometry collision mesh filename=./meshes/R_Ankle.obj scale=1.00000 1.00000 1.00000; visual mesh filename=./meshes/R_Ankle.obj scale=1.00000 1.00000 1.00000
- link right_clavicle_limb: geometry collision mesh filename=./meshes/R_Collar.obj scale=1.00000 1.00000 1.00000; visual mesh filename=./meshes/R_Collar.obj scale=1.00000 1.00000 1.00000
- link right_elbow_limb: geometry collision mesh filename=./meshes/R_Elbow.obj scale=1.00000 1.00000 1.00000; visual mesh filename=./meshes/R_Elbow.obj scale=1.00000 1.00000 1.00000
- link right_foot_limb: geometry collision mesh filename=./meshes/R_Foot.obj scale=1.00000 1.00000 1.00000; visual mesh filename=./meshes/R_Foot.obj scale=1.00000 1.00000 1.00000
- link right_hand_limb: geometry collision mesh filename=./meshes/R_Hand.obj scale=1.00000 1.00000 1.00000; visual mesh filename=./meshes/R_Hand.obj scale=1.00000 1.00000 1.00000
- link right_hip_limb: geometry collision mesh filename=./meshes/R_Hip.obj scale=1.00000 1.00000 1.00000; visual mesh filename=./meshes/R_Hip.obj scale=1.00000 1.00000 1.00000
- link right_knee_limb: geometry collision mesh filename=./meshes/R_Knee.obj scale=1.00000 1.00000 1.00000; visual mesh filename=./meshes/R_Knee.obj scale=1.00000 1.00000 1.00000
- link right_lowarm_limb: geometry collision mesh filename=./meshes/R_Wrist.obj scale=1.00000 1.00000 1.00000; visual mesh filename=./meshes/R_Wrist.obj scale=1.00000 1.00000 1.00000
- link right_shoulder_limb: geometry collision mesh filename=./meshes/R_Shoulder.obj scale=1.00000 1.00000 1.00000; visual mesh filename=./meshes/R_Shoulder.obj scale=1.00000 1.00000 1.00000
- link spine_2_limb: geometry collision mesh filename=./meshes/Spine1.obj scale=1.00000 1.00000 1.00000; visual mesh filename=./meshes/Spine1.obj scale=1.00000 1.00000 1.00000
- link spine_3_limb: geometry collision mesh filename=./meshes/Spine2.obj scale=1.00000 1.00000 1.00000; visual mesh filename=./meshes/Spine2.obj scale=1.00000 1.00000 1.00000
- link spine_4_limb: geometry collision mesh filename=./meshes/Spine3.obj scale=1.00000 1.00000 1.00000; visual mesh filename=./meshes/Spine3.obj scale=1.00000 1.00000 1.00000

Commit message: able to generate working urdf for different people

File: assistive_gym/envs/assets/human/ref_mesh.urdf (robot description, URDF)
Before this commit: robot human, 94 links, 93 joints
Links:
- link head_limb: geometry collision mesh filename=/meshes/Head.obj scale=1.00000 1.00000 1.00000; visual mesh filename=/meshes/Head.obj scale=1.00000 1.00000 1.00000
- link left_ankle_limb: geometry collision mesh filename=/meshes/L_Ankle.obj scale=1.00000 1.00000 1.00000; visual mesh filename=/meshes/L_Ankle.obj scale=1.00000 1.00000 1.00000
- link left_clavicle_limb: geometry collision mesh filename=/meshes/L_Collar.obj scale=1.00000 1.00000 1.00000; visual mesh filename=/meshes/L_Collar.obj scale=1.00000 1.00000 1.00000
- link left_elbow_limb: geometry collision mesh filename=/meshes/L_Elbow.obj scale=1.00000 1.00000 1.00000; visual mesh filename=/meshes/L_Elbow.obj scale=1.00000 1.00000 1.00000
- link left_foot_limb: geometry collision mesh filename=/meshes/L_Foot.obj scale=1.00000 1.00000 1.00000; visual mesh filename=/meshes/L_Foot.obj scale=1.00000 1.00000 1.00000
- link left_hand_limb: geometry collision mesh filename=/meshes/L_Hand.obj scale=1.00000 1.00000 1.00000; visual mesh filename=/meshes/L_Hand.obj scale=1.00000 1.00000 1.00000
- link left_hip_limb: geometry collision mesh filename=/meshes/L_Hip.obj scale=1.00000 1.00000 1.00000; visual mesh filename=/meshes/L_Hip.obj scale=1.00000 1.00000 1.00000
- link left_knee_limb: geometry collision mesh filename=/meshes/L_Knee.obj scale=1.00000 1.00000 1.00000; visual mesh filename=/meshes/L_Knee.obj scale=1.00000 1.00000 1.00000
- link left_lowarm_limb: geometry collision mesh filename=/meshes/L_Wrist.obj scale=1.00000 1.00000 1.00000; visual mesh filename=/meshes/L_Wrist.obj scale=1.00000 1.00000 1.00000
- link left_shoulder_limb: geometry collision mesh filename=/meshes/L_Shoulder.obj scale=1.00000 1.00000 1.00000; visual mesh filename=/meshes/L_Shoulder.obj scale=1.00000 1.00000 1.00000
- link neck_limb: geometry collision mesh filename=/meshes/Neck.obj scale=1.00000 1.00000 1.00000; visual mesh filename=/meshes/Neck.obj scale=1.00000 1.00000 1.00000
- link pelvis_limb: geometry collision mesh filename=/meshes/Pelvis.obj scale=1.00000 1.00000 1.00000; visual mesh filename=/meshes/Pelvis.obj scale=1.00000 1.00000 1.00000
- link right_ankle_limb: geometry collision mesh filename=/meshes/R_Ankle.obj scale=1.00000 1.00000 1.00000; visual mesh filename=/meshes/R_Ankle.obj scale=1.00000 1.00000 1.00000
- link right_clavicle_limb: geometry collision mesh filename=/meshes/R_Collar.obj scale=1.00000 1.00000 1.00000; visual mesh filename=/meshes/R_Collar.obj scale=1.00000 1.00000 1.00000
- link right_elbow_limb: geometry collision mesh filename=/meshes/R_Elbow.obj scale=1.00000 1.00000 1.00000; visual mesh filename=/meshes/R_Elbow.obj scale=1.00000 1.00000 1.00000
- link right_foot_limb: geometry collision mesh filename=/meshes/R_Foot.obj scale=1.00000 1.00000 1.00000; visual mesh filename=/meshes/R_Foot.obj scale=1.00000 1.00000 1.00000
- link right_hand_limb: geometry collision mesh filename=/meshes/R_Hand.obj scale=1.00000 1.00000 1.00000; visual mesh filename=/meshes/R_Hand.obj scale=1.00000 1.00000 1.00000
- link right_hip_limb: geometry collision mesh filename=/meshes/R_Hip.obj scale=1.00000 1.00000 1.00000; visual mesh filename=/meshes/R_Hip.obj scale=1.00000 1.00000 1.00000
- link right_knee_limb: geometry collision mesh filename=/meshes/R_Knee.obj scale=1.00000 1.00000 1.00000; visual mesh filename=/meshes/R_Knee.obj scale=1.00000 1.00000 1.00000
- link right_lowarm_limb: geometry collision mesh filename=/meshes/R_Wrist.obj scale=1.00000 1.00000 1.00000; visual mesh filename=/meshes/R_Wrist.obj scale=1.00000 1.00000 1.00000
- link right_shoulder_limb: geometry collision mesh filename=/meshes/R_Shoulder.obj scale=1.00000 1.00000 1.00000; visual mesh filename=/meshes/R_Shoulder.obj scale=1.00000 1.00000 1.00000
- link spine_2_limb: geometry collision mesh filename=/meshes/Spine1.obj scale=1.00000 1.00000 1.00000; visual mesh filename=/meshes/Spine1.obj scale=1.00000 1.00000 1.00000
- link spine_3_limb: geometry collision mesh filename=/meshes/Spine2.obj scale=1.00000 1.00000 1.00000; visual mesh filename=/meshes/Spine2.obj scale=1.00000 1.00000 1.00000
- link spine_4_limb: geometry collision mesh filename=/meshes/Spine3.obj scale=1.00000 1.00000 1.00000; visual mesh filename=/meshes/Spine3.obj scale=1.00000 1.00000 1.00000
