Commit message: able to offset joint in urdf, but current joint is set to child position - bug

File: test_mesh_joint_child.urdf (robot description, URDF)
Before this commit: robot human, 95 links, 94 joints
Links:
- link head_limb: geometry collision mesh filename=./assistive_gym/envs/assets/human/meshes/Head.obj scale=1.00000 1.00000 1.00000; visual mesh filename=./assistive_gym/envs/assets/human/meshes/Head.obj scale=1.00000 1.00000 1.00000
- link left_ankle_limb: geometry collision mesh filename=./assistive_gym/envs/assets/human/meshes/L_Ankle.obj scale=1.00000 1.00000 1.00000; visual mesh filename=./assistive_gym/envs/assets/human/meshes/L_Ankle.obj scale=1.00000 1.00000 1.00000
- link left_clavicle_rx: geometry collision mesh filename=./assistive_gym/envs/assets/human/meshes/L_Collar.obj scale=1.00000 1.00000 1.00000; visual mesh filename=./assistive_gym/envs/assets/human/meshes/L_Collar.obj scale=1.00000 1.00000 1.00000
- link left_elbow_limb: geometry collision mesh filename=./assistive_gym/envs/assets/human/meshes/L_Elbow.obj scale=1.00000 1.00000 1.00000; visual mesh filename=./assistive_gym/envs/assets/human/meshes/L_Elbow.obj scale=1.00000 1.00000 1.00000
- link left_foot_limb: geometry collision mesh filename=./assistive_gym/envs/assets/human/meshes/L_Foot.obj scale=1.00000 1.00000 1.00000; visual mesh filename=./assistive_gym/envs/assets/human/meshes/L_Foot.obj scale=1.00000 1.00000 1.00000
- link left_hand_limb: geometry collision mesh filename=./assistive_gym/envs/assets/human/meshes/L_Hand.obj scale=1.00000 1.00000 1.00000; visual mesh filename=./assistive_gym/envs/assets/human/meshes/L_Hand.obj scale=1.00000 1.00000 1.00000
- link left_hip_rx: geometry collision mesh filename=./assistive_gym/envs/assets/human/meshes/L_Hip.obj scale=1.00000 1.00000 1.00000; visual mesh filename=./assistive_gym/envs/assets/human/meshes/L_Hip.obj scale=1.00000 1.00000 1.00000
- link left_knee_limb: geometry collision mesh filename=./assistive_gym/envs/assets/human/meshes/L_Knee.obj scale=1.00000 1.00000 1.00000; visual mesh filename=./assistive_gym/envs/assets/human/meshes/L_Knee.obj scale=1.00000 1.00000 1.00000
- link left_lowarm_limb: geometry collision mesh filename=./assistive_gym/envs/assets/human/meshes/L_Wrist.obj scale=1.00000 1.00000 1.00000; visual mesh filename=./assistive_gym/envs/assets/human/meshes/L_Wrist.obj scale=1.00000 1.00000 1.00000
- link left_shoulder_limb: geometry collision mesh filename=./assistive_gym/envs/assets/human/meshes/L_Shoulder.obj scale=1.00000 1.00000 1.00000; visual mesh filename=./assistive_gym/envs/assets/human/meshes/L_Shoulder.obj scale=1.00000 1.00000 1.00000
- link neck_limb: geometry collision mesh filename=./assistive_gym/envs/assets/human/meshes/Neck.obj scale=1.00000 1.00000 1.00000; visual mesh filename=./assistive_gym/envs/assets/human/meshes/Neck.obj scale=1.00000 1.00000 1.00000
- link pelvis_dammy: geometry collision mesh filename=./assistive_gym/envs/assets/human/meshes/Pelvis.obj scale=1.00000 1.00000 1.00000; visual mesh filename=./assistive_gym/envs/assets/human/meshes/Pelvis.obj scale=1.00000 1.00000 1.00000
- link right_ankle_limb: geometry collision mesh filename=./assistive_gym/envs/assets/human/meshes/R_Ankle.obj scale=1.00000 1.00000 1.00000; visual mesh filename=./assistive_gym/envs/assets/human/meshes/R_Ankle.obj scale=1.00000 1.00000 1.00000
- link right_clavicle_rx: geometry collision mesh filename=./assistive_gym/envs/assets/human/meshes/R_Collar.obj scale=1.00000 1.00000 1.00000; visual mesh filename=./assistive_gym/envs/assets/human/meshes/R_Collar.obj scale=1.00000 1.00000 1.00000
- link right_elbow_limb: geometry collision mesh filename=./assistive_gym/envs/assets/human/meshes/R_Elbow.obj scale=1.00000 1.00000 1.00000; visual mesh filename=./assistive_gym/envs/assets/human/meshes/R_Elbow.obj scale=1.00000 1.00000 1.00000
- link right_foot_limb: geometry collision mesh filename=./assistive_gym/envs/assets/human/meshes/R_Foot.obj scale=1.00000 1.00000 1.00000; visual mesh filename=./assistive_gym/envs/assets/human/meshes/R_Foot.obj scale=1.00000 1.00000 1.00000
- link right_hand_limb: geometry collision mesh filename=./assistive_gym/envs/assets/human/meshes/R_Hand.obj scale=1.00000 1.00000 1.00000; visual mesh filename=./assistive_gym/envs/assets/human/meshes/R_Hand.obj scale=1.00000 1.00000 1.00000
- link right_hip_rx: geometry collision mesh filename=./assistive_gym/envs/assets/human/meshes/R_Hip.obj scale=1.00000 1.00000 1.00000; visual mesh filename=./assistive_gym/envs/assets/human/meshes/R_Hip.obj scale=1.00000 1.00000 1.00000
- link right_knee_limb: geometry collision mesh filename=./assistive_gym/envs/assets/human/meshes/R_Knee.obj scale=1.00000 1.00000 1.00000; visual mesh filename=./assistive_gym/envs/assets/human/meshes/R_Knee.obj scale=1.00000 1.00000 1.00000
- link right_lowarm_limb: geometry collision mesh filename=./assistive_gym/envs/assets/human/meshes/R_Wrist.obj scale=1.00000 1.00000 1.00000; visual mesh filename=./assistive_gym/envs/assets/human/meshes/R_Wrist.obj scale=1.00000 1.00000 1.00000
- link right_shoulder_limb: geometry collision mesh filename=./assistive_gym/envs/assets/human/meshes/R_Shoulder.obj scale=1.00000 1.00000 1.00000; visual mesh filename=./assistive_gym/envs/assets/human/meshes/R_Shoulder.obj scale=1.00000 1.00000 1.00000
- link spine_2_limb: geometry collision mesh filename=./assistive_gym/envs/assets/human/meshes/Spine1.obj scale=1.00000 1.00000 1.00000; visual mesh filename=./assistive_gym/envs/assets/human/meshes/Spine1.obj scale=1.00000 1.00000 1.00000
- link spine_3_limb: geometry collision mesh filename=./assistive_gym/envs/assets/human/meshes/Spine2.obj scale=1.00000 1.00000 1.00000; visual mesh filename=./assistive_gym/envs/assets/human/meshes/Spine2.obj scale=1.00000 1.00000 1.00000
- link spine_4_limb: geometry collision mesh filename=./assistive_gym/envs/assets/human/meshes/Spine3.obj scale=1.00000 1.00000 1.00000; visual mesh filename=./assistive_gym/envs/assets/human/meshes/Spine3.obj scale=1.00000 1.00000 1.00000
Joints:
- joint left_ankle_rzdammy: origin xyz=0.00000 0.00000 0.00000 rpy=0.00000 -0.00000 0.00000 -> xyz=0.04105 -0.06029 0.12204 rpy=0.00000 -0.00000 0.00000
- joint left_clavicle_rx: origin xyz=0.00000 0.00000 0.00000 rpy=0.00000 -0.00000 0.00000 -> xyz=0.07170 0.11400 -0.01890 rpy=0.00000 -0.00000 0.00000
- joint left_clavicle_rzdammy: origin xyz=0.00000 0.00000 0.00000 rpy=0.00000 -0.00000 0.00000 -> xyz=0.12292 0.04521 -0.01905 rpy=0.00000 -0.00000 0.00000
- joint left_elbow_rzdammy: origin xyz=0.00000 0.00000 0.00000 rpy=0.00000 -0.00000 0.00000 -> xyz=0.26571 0.01270 -0.00737 rpy=0.00000 -0.00000 0.00000
- joint left_heel: origin xyz=-0.13000 0.00510 0.00000 rpy=0.00000 -0.00000 0.00000 -> xyz=0.00000 0.00000 0.00000 rpy=0.00000 -0.00000 0.00000
- joint left_hip_rx: origin xyz=0.00000 0.00000 0.00000 rpy=0.00000 -0.00000 0.00000 -> xyz=0.05858 -0.08228 -0.01766 rpy=0.00000 -0.00000 0.00000
- joint left_hip_rzdammy: origin xyz=0.00000 0.00000 0.00000 rpy=0.00000 -0.00000 0.00000 -> xyz=0.04345 -0.38647 0.00804 rpy=0.00000 -0.00000 0.00000
- joint left_knee_rzdammy: origin xyz=0.00000 0.00000 0.00000 rpy=0.00000 -0.00000 0.00000 -> xyz=-0.01479 -0.42687 -0.03743 rpy=0.00000 -0.00000 0.00000
- joint left_lowarm_rzdammy: origin xyz=0.00000 0.00000 0.00000 rpy=0.00000 -0.00000 0.00000 -> xyz=0.08669 -0.01064 -0.01559 rpy=0.00000 -0.00000 0.00000
- joint left_shoulder_rzdammy: origin xyz=0.00000 0.00000 0.00000 rpy=0.00000 -0.00000 0.00000 -> xyz=0.25533 -0.01565 -0.02295 rpy=0.00000 -0.00000 0.00000
- joint left_toe: origin xyz=0.01100 0.00000 -0.01000 rpy=1.57080 -0.00000 0.00000 -> xyz=0.00000 0.00000 0.00000 rpy=1.57080 -0.00000 0.00000
- joint neck_rzdammy: origin xyz=0.00000 0.00000 0.00000 rpy=0.00000 -0.00000 0.00000 -> xyz=0.01011 0.08894 0.05041 rpy=0.00000 -0.00000 0.00000
- joint pelvis_dammy: origin xyz=0.00000 0.00000 0.00000 rpy=0.00000 0 0 -> xyz=0.00000 0.00000 0.00000 rpy=0.00000 -0.00000 0.00000
- joint right_ankle_rzdammy: origin xyz=0.00000 0.00000 0.00000 rpy=0.00000 -0.00000 0.00000 -> xyz=-0.03484 -0.06211 0.13032 rpy=0.00000 -0.00000 0.00000
- joint right_clavicle_rx: origin xyz=0.00000 0.00000 0.00000 rpy=0.00000 -0.00000 0.00000 -> xyz=-0.08295 0.11247 -0.02371 rpy=0.00000 -0.00000 0.00000
- joint right_clavicle_rzdammy: origin xyz=0.00000 0.00000 0.00000 rpy=0.00000 -0.00000 0.00000 -> xyz=-0.11323 0.04685 -0.00847 rpy=0.00000 -0.00000 0.00000
- joint right_elbow_rzdammy: origin xyz=0.00000 0.00000 0.00000 rpy=0.00000 -0.00000 0.00000 -> xyz=-0.26911 0.00679 -0.00603 rpy=0.00000 -0.00000 0.00000
- joint right_heel: origin xyz=-0.13000 -0.00510 0.00000 rpy=0.00000 -0.00000 0.00000 -> xyz=0.00000 0.00000 0.00000 rpy=0.00000 -0.00000 0.00000
- joint right_hip_rx: origin xyz=0.00000 0.00000 0.00000 rpy=0.00000 -0.00000 0.00000 -> xyz=-0.06031 -0.09051 -0.01354 rpy=0.00000 -0.00000 0.00000
- joint right_hip_rzdammy: origin xyz=0.00000 0.00000 0.00000 rpy=0.00000 -0.00000 0.00000 -> xyz=-0.04326 -0.38369 -0.00484 rpy=0.00000 -0.00000 0.00000
- joint right_knee_rzdammy: origin xyz=0.00000 0.00000 0.00000 rpy=0.00000 -0.00000 0.00000 -> xyz=0.01906 -0.42005 -0.03456 rpy=0.00000 -0.00000 0.00000
- joint right_lowarm_rzdammy: origin xyz=0.00000 0.00000 0.00000 rpy=0.00000 -0.00000 0.00000 -> xyz=-0.08875 -0.00865 -0.01011 rpy=0.00000 -0.00000 0.00000
- joint right_shoulder_rzdammy: origin xyz=0.00000 0.00000 0.00000 rpy=0.00000 -0.00000 0.00000 -> xyz=-0.26013 -0.01437 -0.03127 rpy=0.00000 -0.00000 0.00000
- joint right_toe: origin xyz=0.01100 0.00000 -0.01000 rpy=1.57080 -0.00000 0.00000 -> xyz=0.00000 0.00000 0.00000 rpy=1.57080 -0.00000 0.00000
- joint spine_2_rzdammy: origin xyz=0.00000 0.00000 0.00000 rpy=0.00000 -0.00000 0.00000 -> xyz=0.00449 0.13796 0.02682 rpy=0.00000 -0.00000 0.00000
- joint spine_3_rzdammy: origin xyz=0.00000 0.00000 0.00000 rpy=0.00000 -0.00000 0.00000 -> xyz=-0.00226 0.05603 0.00286 rpy=0.00000 -0.00000 0.00000
- joint spine_4_rzdammy: origin xyz=0.00000 0.00000 0.00000 rpy=0.00000 -0.00000 0.00000 -> xyz=-0.08295 0.11247 -0.02371 rpy=0.00000 -0.00000 0.00000
