Commit message: it works

File: ref_mesh.urdf (robot description, URDF)
Before this commit: robot human, 97 links, 96 joints
Links:
- removed link pelvis
- removed link pelvis_dammy
- added link left_clavicle_limb, mass 0.00001; collision mesh filename=././assistive_gym/envs/assets/human/meshes/L_Collar.obj scale=1.00000 1.00000 1.00000; visual mesh filename=././assistive_gym/envs/assets/human/meshes/L_Collar.obj scale=1.00000 1.00000 1.00000
- added link pelvis_limb, mass 0.00001; collision mesh filename=assistive_gym/envs/assets/human/meshes/Pelvis.obj scale=1.00000 1.00000 1.00000; visual mesh filename=assistive_gym/envs/assets/human/meshes/Pelvis.obj scale=1.00000 1.00000 1.00000
- added link right_clavicle_limb, mass 0.00001; collision mesh filename=././assistive_gym/envs/assets/human/meshes/R_Collar.obj scale=1.00000 1.00000 1.00000; visual mesh filename=././assistive_gym/envs/assets/human/meshes/R_Collar.obj scale=1.00000 1.00000 1.00000
- link head_limb: geometry collision mesh filename=././assistive_gym/envs/assets/human/meshes/Head.obj scale=1.00000 1.00000 1.00000; visual mesh filename=././assistive_gym/envs/assets/human/meshes/Head.obj scale=1.00000 1.00000 1.00000
- link left_ankle_limb: geometry collision mesh filename=././assistive_gym/envs/assets/human/meshes/L_Ankle.obj scale=1.00000 1.00000 1.00000; visual mesh filename=././assistive_gym/envs/assets/human/meshes/L_Ankle.obj scale=1.00000 1.00000 1.00000
- link left_clavicle_rx: geometry collision sphere radius=0.00000; visual sphere radius=0.00000
- link left_elbow_limb: geometry collision mesh filename=././assistive_gym/envs/assets/human/meshes/L_Elbow.obj scale=1.00000 1.00000 1.00000; visual mesh filename=././assistive_gym/envs/assets/human/meshes/L_Elbow.obj scale=1.00000 1.00000 1.00000
- link left_foot_limb: geometry collision mesh filename=././assistive_gym/envs/assets/human/meshes/L_Foot.obj scale=1.00000 1.00000 1.00000; visual mesh filename=././assistive_gym/envs/assets/human/meshes/L_Foot.obj scale=1.00000 1.00000 1.00000
- link left_hand_limb: geometry collision mesh filename=././assistive_gym/envs/assets/human/meshes/L_Hand.obj scale=1.00000 1.00000 1.00000; visual mesh filename=././assistive_gym/envs/assets/human/meshes/L_Hand.obj scale=1.00000 1.00000 1.00000
- link left_hip_limb: geometry collision mesh filename=././assistive_gym/envs/assets/human/meshes/L_Hip.obj scale=1.00000 1.00000 1.00000; visual mesh filename=././assistive_gym/envs/assets/human/meshes/L_Hip.obj scale=1.00000 1.00000 1.00000
- link left_knee_limb: geometry collision mesh filename=././assistive_gym/envs/assets/human/meshes/L_Knee.obj scale=1.00000 1.00000 1.00000; visual mesh filename=././assistive_gym/envs/assets/human/meshes/L_Knee.obj scale=1.00000 1.00000 1.00000
- link left_lowarm_limb: geometry collision mesh filename=././assistive_gym/envs/assets/human/meshes/L_Wrist.obj scale=1.00000 1.00000 1.00000; visual mesh filename=././assistive_gym/envs/assets/human/meshes/L_Wrist.obj scale=1.00000 1.00000 1.00000
- link left_shoulder_limb: geometry collision mesh filename=././assistive_gym/envs/assets/human/meshes/L_Shoulder.obj scale=1.00000 1.00000 1.00000; visual mesh filename=././assistive_gym/envs/assets/human/meshes/L_Shoulder.obj scale=1.00000 1.00000 1.00000
- link neck_limb: geometry collision mesh filename=././assistive_gym/envs/assets/human/meshes/Neck.obj scale=1.00000 1.00000 1.00000; visual mesh filename=././assistive_gym/envs/assets/human/meshes/Neck.obj scale=1.00000 1.00000 1.00000
- link right_ankle_limb: geometry collision mesh filename=././assistive_gym/envs/assets/human/meshes/R_Ankle.obj scale=1.00000 1.00000 1.00000; visual mesh filename=././assistive_gym/envs/assets/human/meshes/R_Ankle.obj scale=1.00000 1.00000 1.00000
- link right_clavicle_rx: geometry collision sphere radius=0.00000; visual sphere radius=0.00000
- link right_elbow_limb: geometry collision mesh filename=././assistive_gym/envs/assets/human/meshes/R_Elbow.obj scale=1.00000 1.00000 1.00000; visual mesh filename=././assistive_gym/envs/assets/human/meshes/R_Elbow.obj scale=1.00000 1.00000 1.00000
- link right_foot_limb: geometry collision mesh filename=././assistive_gym/envs/assets/human/meshes/R_Foot.obj scale=1.00000 1.00000 1.00000; visual mesh filename=././assistive_gym/envs/assets/human/meshes/R_Foot.obj scale=1.00000 1.00000 1.00000
- link right_hand_limb: geometry collision mesh filename=././assistive_gym/envs/assets/human/meshes/R_Hand.obj scale=1.00000 1.00000 1.00000; visual mesh filename=././assistive_gym/envs/assets/human/meshes/R_Hand.obj scale=1.00000 1.00000 1.00000
- link right_hip_limb: geometry collision mesh filename=././assistive_gym/envs/assets/human/meshes/R_Hip.obj scale=1.00000 1.00000 1.00000; visual mesh filename=././assistive_gym/envs/assets/human/meshes/R_Hip.obj scale=1.00000 1.00000 1.00000
- link right_knee_limb: geometry collision mesh filename=././assistive_gym/envs/assets/human/meshes/R_Knee.obj scale=1.00000 1.00000 1.00000; visual mesh filename=././assistive_gym/envs/assets/human/meshes/R_Knee.obj scale=1.00000 1.00000 1.00000
- link right_lowarm_limb: geometry collision mesh filename=././assistive_gym/envs/assets/human/meshes/R_Wrist.obj scale=1.00000 1.00000 1.00000; visual mesh filename=././assistive_gym/envs/assets/human/meshes/R_Wrist.obj scale=1.00000 1.00000 1.00000
- link right_shoulder_limb: geometry collision mesh filename=././assistive_gym/envs/assets/human/meshes/R_Shoulder.obj scale=1.00000 1.00000 1.00000; visual mesh filename=././assistive_gym/envs/assets/human/meshes/R_Shoulder.obj scale=1.00000 1.00000 1.00000
- link spine_2_limb: geometry collision mesh filename=././assistive_gym/envs/assets/human/meshes/Spine1.obj scale=1.00000 1.00000 1.00000; visual mesh filename=././assistive_gym/envs/assets/human/meshes/Spine1.obj scale=1.00000 1.00000 1.00000
- link spine_3_limb: geometry collision mesh filename=././assistive_gym/envs/assets/human/meshes/Spine2.obj scale=1.00000 1.00000 1.00000; visual mesh filename=././assistive_gym/envs/assets/human/meshes/Spine2.obj scale=1.00000 1.00000 1.00000
- link spine_4_limb: geometry collision mesh filename=././assistive_gym/envs/assets/human/meshes/Spine3.obj scale=1.00000 1.00000 1.00000; visual mesh filename=././assistive_gym/envs/assets/human/meshes/Spine3.obj scale=1.00000 1.00000 1.00000
Joints:
- removed joint pelvis_dammy
- removed joint pelvisdammy
- added joint head_rzdammy: type fixed, parent head_rz, child head_limb, origin xyz=0.00000 0.00000 0.00000 rpy=0.00000 -0.00000 0.00000, axis 1.00000 0.00000 0.00000
- added joint left_hand_rzdammy: type revolute, parent left_hand_rz, child left_hand_limb, origin xyz=0.00000 0.00000 0.00000 rpy=0.00000 -0.00000 0.00000, axis 1.00000 0.00000 0.00000, limit lower=-2.50000 upper=2.50000 effort=1000.00000 velocity=0.50000
- added joint right_hand_rzdammy: type revolute, parent right_hand_rz, child right_hand_limb, origin xyz=0.00000 0.00000 0.00000 rpy=0.00000 -0.00000 0.00000, axis 1.00000 0.00000 0.00000, limit lower=-2.50000 upper=2.50000 effort=1000.00000 velocity=0.50000
- joint head_rx: origin xyz=0.00000 0.00000 0.00000 rpy=0.00000 -0.00000 0.00000 -> xyz=0.01011 0.08894 0.05041 rpy=0.00000 -0.00000 0.00000; parent head_limb -> neck_limb
- joint left_ankle_rx: origin xyz=0.00000 0.00000 0.00000 rpy=0.00000 -0.00000 0.00000 -> xyz=-0.01479 -0.42687 -0.03743 rpy=0.00000 -0.00000 0.00000
- joint left_ankle_rzdammy: origin xyz=0.04105 -0.06029 0.12204 rpy=0.00000 -0.00000 0.00000 -> xyz=0.00000 0.00000 0.00000 rpy=0.00000 -0.00000 0.00000
- joint left_clavicle_rx: parent spine_4_rz -> spine_4_limb
- joint left_clavicle_rzdammy: child left_shoulder_limb -> left_clavicle_limb; origin xyz=0.12292 0.04521 -0.01905 rpy=0.00000 -0.00000 0.00000 -> xyz=0.00000 0.00000 0.00000 rpy=0.00000 -0.00000 0.00000
- joint left_elbow_rx: origin xyz=0.00000 0.00000 0.00000 rpy=0.00000 -0.00000 0.00000 -> xyz=0.25533 -0.01565 -0.02295 rpy=0.00000 -0.00000 0.00000; parent left_elbow_limb -> left_shoulder_limb
- joint left_elbow_rzdammy: child left_lowarm_limb -> left_elbow_limb; origin xyz=0.26571 0.01270 -0.00737 rpy=0.00000 -0.00000 0.00000 -> xyz=0.00000 0.00000 0.00000 rpy=0.00000 -0.00000 0.00000
- joint left_foot_rx: origin xyz=0.00000 0.00000 0.00000 rpy=0.00000 -0.00000 0.00000 -> xyz=0.04105 -0.06029 0.12204 rpy=0.00000 -0.00000 0.00000
- joint left_foot_rzdammy: axis 1.00000 0.00000 0.00000 -> 0.00000 0.00000 0.00000
- joint left_hand_rx: origin xyz=0.00000 0.00000 0.00000 rpy=0.00000 -0.00000 0.00000 -> xyz=0.08669 -0.01064 -0.01559 rpy=0.00000 -0.00000 0.00000; parent left_hand_limb -> left_lowarm_limb
- joint left_hip_rx: origin xyz=0.00000 0.00000 0.00000 rpy=0.00000 -0.00000 0.00000 -> xyz=0.05858 -0.08228 -0.01766 rpy=0.00000 -0.00000 0.00000; parent pelvis_dammy -> pelvis_limb
- joint left_hip_rzdammy: origin xyz=0.04345 -0.38647 0.00804 rpy=0.00000 -0.00000 0.00000 -> xyz=0.00000 0.00000 0.00000 rpy=0.00000 -0.00000 0.00000
- joint left_knee_rx: origin xyz=0.00000 0.00000 0.00000 rpy=0.00000 -0.00000 0.00000 -> xyz=0.04345 -0.38647 0.00804 rpy=0.00000 -0.00000 0.00000
- joint left_knee_rzdammy: origin xyz=-0.01479 -0.42687 -0.03743 rpy=0.00000 -0.00000 0.00000 -> xyz=0.00000 0.00000 0.00000 rpy=0.00000 -0.00000 0.00000
- joint left_lowarm_rx: origin xyz=0.00000 0.00000 0.00000 rpy=0.00000 -0.00000 0.00000 -> xyz=0.26571 0.01270 -0.00737 rpy=0.00000 -0.00000 0.00000; parent left_lowarm_limb -> left_elbow_limb
- joint left_lowarm_rzdammy: child left_hand_limb -> left_lowarm_limb; origin xyz=0.08669 -0.01064 -0.01559 rpy=0.00000 -0.00000 0.00000 -> xyz=0.00000 0.00000 0.00000 rpy=0.00000 -0.00000 0.00000
- joint left_shoulder_rx: origin xyz=0.00000 0.00000 0.00000 rpy=0.00000 -0.00000 0.00000 -> xyz=0.12292 0.04521 -0.01905 rpy=0.00000 -0.00000 0.00000; parent left_shoulder_limb -> left_clavicle_limb
- joint left_shoulder_rzdammy: child left_elbow_limb -> left_shoulder_limb; origin xyz=0.25533 -0.01565 -0.02295 rpy=0.00000 -0.00000 0.00000 -> xyz=0.00000 0.00000 0.00000 rpy=0.00000 -0.00000 0.00000
- joint neck_rx: origin xyz=0.00000 0.00000 0.00000 rpy=0.00000 -0.00000 0.00000 -> xyz=-0.01339 0.21164 -0.03347 rpy=0.00000 -0.00000 0.00000; parent neck_limb -> spine_4_limb
- joint neck_rzdammy: child head_limb -> neck_limb; origin xyz=0.01011 0.08894 0.05041 rpy=0.00000 -0.00000 0.00000 -> xyz=0.00000 0.00000 0.00000 rpy=0.00000 -0.00000 0.00000
- joint pelvis: child pelvis -> pelvis_limb
- joint right_ankle_rx: origin xyz=0.00000 0.00000 0.00000 rpy=0.00000 -0.00000 0.00000 -> xyz=0.01906 -0.42005 -0.03456 rpy=0.00000 -0.00000 0.00000
- joint right_ankle_rzdammy: origin xyz=-0.03484 -0.06211 0.13032 rpy=0.00000 -0.00000 0.00000 -> xyz=0.00000 0.00000 0.00000 rpy=0.00000 -0.00000 0.00000
- joint right_clavicle_rx: parent spine_4_rz -> spine_4_limb
- joint right_clavicle_rzdammy: child right_shoulder_limb -> right_clavicle_limb; origin xyz=-0.11323 0.04685 -0.00847 rpy=0.00000 -0.00000 0.00000 -> xyz=0.00000 0.00000 0.00000 rpy=0.00000 -0.00000 0.00000
- joint right_elbow_rx: origin xyz=0.00000 0.00000 0.00000 rpy=0.00000 -0.00000 0.00000 -> xyz=-0.26013 -0.01437 -0.03127 rpy=0.00000 -0.00000 0.00000; parent right_elbow_limb -> right_shoulder_limb
- joint right_elbow_rzdammy: child right_lowarm_limb -> right_elbow_limb; origin xyz=-0.26911 0.00679 -0.00603 rpy=0.00000 -0.00000 0.00000 -> xyz=0.00000 0.00000 0.00000 rpy=0.00000 -0.00000 0.00000
- joint right_foot_rx: origin xyz=0.00000 0.00000 0.00000 rpy=0.00000 -0.00000 0.00000 -> xyz=-0.03484 -0.06211 0.13032 rpy=0.00000 -0.00000 0.00000
- joint right_foot_rzdammy: axis 1.00000 0.00000 0.00000 -> 0.00000 0.00000 0.00000
- joint right_hand_rx: origin xyz=0.00000 0.00000 0.00000 rpy=0.00000 -0.00000 0.00000 -> xyz=-0.08875 -0.00865 -0.01011 rpy=0.00000 -0.00000 0.00000; parent right_hand_limb -> right_lowarm_limb
- joint right_hip_rx: origin xyz=0.00000 0.00000 0.00000 rpy=0.00000 -0.00000 0.00000 -> xyz=-0.06031 -0.09051 -0.01354 rpy=0.00000 -0.00000 0.00000; parent pelvis_dammy -> pelvis_limb
- joint right_hip_rzdammy: origin xyz=-0.04326 -0.38369 -0.00484 rpy=0.00000 -0.00000 0.00000 -> xyz=0.00000 0.00000 0.00000 rpy=0.00000 -0.00000 0.00000
- joint right_knee_rx: origin xyz=0.00000 0.00000 0.00000 rpy=0.00000 -0.00000 0.00000 -> xyz=-0.04326 -0.38369 -0.00484 rpy=0.00000 -0.00000 0.00000
- joint right_knee_rzdammy: origin xyz=0.01906 -0.42005 -0.03456 rpy=0.00000 -0.00000 0.00000 -> xyz=0.00000 0.00000 0.00000 rpy=0.00000 -0.00000 0.00000
- joint right_lowarm_rx: origin xyz=0.00000 0.00000 0.00000 rpy=0.00000 -0.00000 0.00000 -> xyz=-0.26911 0.00679 -0.00603 rpy=0.00000 -0.00000 0.00000; parent right_lowarm_limb -> right_elbow_limb
- joint right_lowarm_rzdammy: child right_hand_limb -> right_lowarm_limb; origin xyz=-0.08875 -0.00865 -0.01011 rpy=0.00000 -0.00000 0.00000 -> xyz=0.00000 0.00000 0.00000 rpy=0.00000 -0.00000 0.00000
- joint right_shoulder_rx: origin xyz=0.00000 0.00000 0.00000 rpy=0.00000 -0.00000 0.00000 -> xyz=-0.11323 0.04685 -0.00847 rpy=0.00000 -0.00000 0.00000; parent right_shoulder_limb -> right_clavicle_limb
- joint right_shoulder_rzdammy: child right_elbow_limb -> right_shoulder_limb; origin xyz=-0.26013 -0.01437 -0.03127 rpy=0.00000 -0.00000 0.00000 -> xyz=0.00000 0.00000 0.00000 rpy=0.00000 -0.00000 0.00000
- joint spine_2_rx: origin xyz=0.00000 0.00000 0.00000 rpy=0.00000 -0.00000 0.00000 -> xyz=0.00444 0.12440 -0.03839 rpy=0.00000 -0.00000 0.00000; parent spine_2_limb -> pelvis_limb
- joint spine_2_rzdammy: child spine_3_limb -> spine_2_limb; origin xyz=0.00449 0.13796 0.02682 rpy=0.00000 -0.00000 0.00000 -> xyz=0.00000 0.00000 0.00000 rpy=0.00000 -0.00000 0.00000
- joint spine_3_rx: origin xyz=0.00000 0.00000 0.00000 rpy=0.00000 -0.00000 0.00000 -> xyz=0.00449 0.13796 0.02682 rpy=0.00000 -0.00000 0.00000; parent spine_3_limb -> spine_2_limb
- joint spine_3_rzdammy: child spine_4_limb -> spine_3_limb; origin xyz=-0.00226 0.05603 0.00286 rpy=0.00000 -0.00000 0.00000 -> xyz=0.00000 0.00000 0.00000 rpy=0.00000 -0.00000 0.00000
- joint spine_4_rx: origin xyz=0.00000 0.00000 0.00000 rpy=0.00000 -0.00000 0.00000 -> xyz=-0.00226 0.05603 0.00286 rpy=0.00000 -0.00000 0.00000; parent spine_4_limb -> spine_3_limb
- joint spine_4_rzdammy: child neck_limb -> spine_4_limb; origin xyz=-0.08295 0.11247 -0.02371 rpy=0.00000 -0.00000 0.00000 -> xyz=0.00000 0.00000 0.00000 rpy=0.00000 -0.00000 0.00000
