Commit message: clean code. fix bug with urdf. fix euler conversion for pose angle

File: ref_mesh.urdf (robot description, URDF)
Before this commit: robot human, 98 links, 97 joints
Links:
- link head_limb: mass 1.00000 -> 2.00000; geometry collision mesh filename=./././assistive_gym/envs/assets/human/meshes/Head.obj scale=1.00000 1.00000 1.00000; visual mesh filename=./././assistive_gym/envs/assets/human/meshes/Head.obj scale=1.00000 1.00000 1.00000
- link left_ankle_limb: geometry collision mesh filename=./././assistive_gym/envs/assets/human/meshes/L_Ankle.obj scale=1.00000 1.00000 1.00000; visual mesh filename=./././assistive_gym/envs/assets/human/meshes/L_Ankle.obj scale=1.00000 1.00000 1.00000
- link left_clavicle_limb: mass 0.00001 -> 2.00000; geometry collision mesh filename=./././assistive_gym/envs/assets/human/meshes/L_Collar.obj scale=1.00000 1.00000 1.00000; visual mesh filename=./././assistive_gym/envs/assets/human/meshes/L_Collar.obj scale=1.00000 1.00000 1.00000
- link left_elbow_limb: mass 1.00000 -> 2.00000; geometry collision mesh filename=./././assistive_gym/envs/assets/human/meshes/L_Elbow.obj scale=1.00000 1.00000 1.00000; visual mesh filename=./././assistive_gym/envs/assets/human/meshes/L_Elbow.obj scale=1.00000 1.00000 1.00000
- link left_foot_limb: mass 1.00000 -> 2.00000; geometry collision mesh filename=./././assistive_gym/envs/assets/human/meshes/L_Foot.obj scale=1.00000 1.00000 1.00000; visual mesh filename=./././assistive_gym/envs/assets/human/meshes/L_Foot.obj scale=1.00000 1.00000 1.00000
- link left_hand_limb: mass 0.50000 -> 2.00000; geometry collision mesh filename=./././assistive_gym/envs/assets/human/meshes/L_Hand.obj scale=1.00000 1.00000 1.00000; visual mesh filename=./././assistive_gym/envs/assets/human/meshes/L_Hand.obj scale=1.00000 1.00000 1.00000
- link left_hip_limb: mass 0.00001 -> 2.00000; geometry collision mesh filename=./././assistive_gym/envs/assets/human/meshes/L_Hip.obj scale=1.00000 1.00000 1.00000; visual mesh filename=./././assistive_gym/envs/assets/human/meshes/L_Hip.obj scale=1.00000 1.00000 1.00000
- link left_knee_limb: geometry collision mesh filename=./././assistive_gym/envs/assets/human/meshes/L_Knee.obj scale=1.00000 1.00000 1.00000; visual mesh filename=./././assistive_gym/envs/assets/human/meshes/L_Knee.obj scale=1.00000 1.00000 1.00000
- link left_lowarm_limb: mass 1.00000 -> 2.00000; geometry collision mesh filename=./././assistive_gym/envs/assets/human/meshes/L_Wrist.obj scale=1.00000 1.00000 1.00000; visual mesh filename=./././assistive_gym/envs/assets/human/meshes/L_Wrist.obj scale=1.00000 1.00000 1.00000
- link left_shoulder_limb: mass 1.00000 -> 2.00000; geometry collision mesh filename=./././assistive_gym/envs/assets/human/meshes/L_Shoulder.obj scale=1.00000 1.00000 1.00000; visual mesh filename=./././assistive_gym/envs/assets/human/meshes/L_Shoulder.obj scale=1.00000 1.00000 1.00000
- link neck_limb: mass 1.00000 -> 2.00000; geometry collision mesh filename=./././assistive_gym/envs/assets/human/meshes/Neck.obj scale=1.00000 1.00000 1.00000; visual mesh filename=./././assistive_gym/envs/assets/human/meshes/Neck.obj scale=1.00000 1.00000 1.00000
- link pelvis_limb: mass 0.00001 -> 2.00000; geometry collision mesh filename=./assistive_gym/envs/assets/human/meshes/Pelvis.obj scale=1.00000 1.00000 1.00000; visual mesh filename=./assistive_gym/envs/assets/human/meshes/Pelvis.obj scale=1.00000 1.00000 1.00000
- link right_ankle_limb: geometry collision mesh filename=./././assistive_gym/envs/assets/human/meshes/R_Ankle.obj scale=1.00000 1.00000 1.00000; visual mesh filename=./././assistive_gym/envs/assets/human/meshes/R_Ankle.obj scale=1.00000 1.00000 1.00000
- link right_clavicle_limb: mass 0.00001 -> 2.00000; geometry collision mesh filename=./././assistive_gym/envs/assets/human/meshes/R_Collar.obj scale=1.00000 1.00000 1.00000; visual mesh filename=./././assistive_gym/envs/assets/human/meshes/R_Collar.obj scale=1.00000 1.00000 1.00000
- link right_elbow_limb: mass 1.00000 -> 2.00000; geometry collision mesh filename=./././assistive_gym/envs/assets/human/meshes/R_Elbow.obj scale=1.00000 1.00000 1.00000; visual mesh filename=./././assistive_gym/envs/assets/human/meshes/R_Elbow.obj scale=1.00000 1.00000 1.00000
- link right_foot_limb: mass 1.00000 -> 2.00000; geometry collision mesh filename=./././assistive_gym/envs/assets/human/meshes/R_Foot.obj scale=1.00000 1.00000 1.00000; visual mesh filename=./././assistive_gym/envs/assets/human/meshes/R_Foot.obj scale=1.00000 1.00000 1.00000
- link right_hand_limb: mass 0.50000 -> 2.00000; geometry collision mesh filename=./././assistive_gym/envs/assets/human/meshes/R_Hand.obj scale=1.00000 1.00000 1.00000; visual mesh filename=./././assistive_gym/envs/assets/human/meshes/R_Hand.obj scale=1.00000 1.00000 1.00000
- link right_hip_limb: mass 0.00001 -> 2.00000; geometry collision mesh filename=./././assistive_gym/envs/assets/human/meshes/R_Hip.obj scale=1.00000 1.00000 1.00000; visual mesh filename=./././assistive_gym/envs/assets/human/meshes/R_Hip.obj scale=1.00000 1.00000 1.00000
- link right_knee_limb: geometry collision mesh filename=./././assistive_gym/envs/assets/human/meshes/R_Knee.obj scale=1.00000 1.00000 1.00000; visual mesh filename=./././assistive_gym/envs/assets/human/meshes/R_Knee.obj scale=1.00000 1.00000 1.00000
- link right_lowarm_limb: mass 1.00000 -> 2.00000; geometry collision mesh filename=./././assistive_gym/envs/assets/human/meshes/R_Wrist.obj scale=1.00000 1.00000 1.00000; visual mesh filename=./././assistive_gym/envs/assets/human/meshes/R_Wrist.obj scale=1.00000 1.00000 1.00000
- link right_shoulder_limb: mass 1.00000 -> 2.00000; geometry collision mesh filename=./././assistive_gym/envs/assets/human/meshes/R_Shoulder.obj scale=1.00000 1.00000 1.00000; visual mesh filename=./././assistive_gym/envs/assets/human/meshes/R_Shoulder.obj scale=1.00000 1.00000 1.00000
- link spine_2_limb: geometry collision mesh filename=./././assistive_gym/envs/assets/human/meshes/Spine1.obj scale=1.00000 1.00000 1.00000; visual mesh filename=./././assistive_gym/envs/assets/human/meshes/Spine1.obj scale=1.00000 1.00000 1.00000
- link spine_3_limb: geometry collision mesh filename=./././assistive_gym/envs/assets/human/meshes/Spine2.obj scale=1.00000 1.00000 1.00000; visual mesh filename=./././assistive_gym/envs/assets/human/meshes/Spine2.obj scale=1.00000 1.00000 1.00000
- link spine_4_limb: geometry collision mesh filename=./././assistive_gym/envs/assets/human/meshes/Spine3.obj scale=1.00000 1.00000 1.00000; visual mesh filename=./././assistive_gym/envs/assets/human/meshes/Spine3.obj scale=1.00000 1.00000 1.00000
Joints:
- joint head_rx: origin xyz=0.01011 0.08894 0.05041 rpy=0.00000 -0.00000 0.00000 -> xyz=0.01011 0.08894 0.05041 rpy=0.00000 0.0000 0.00000
- joint head_ry: origin xyz=0.00000 0.00000 0.00000 rpy=0.00000 -0.00000 0.00000 -> xyz=0.00000 0.00000 0.00000 rpy=0.00000 0.0000 0.00000
- joint head_rz: origin xyz=0.00000 0.00000 0.00000 rpy=0.00000 -0.00000 0.00000 -> xyz=0.00000 0.00000 0.00000 rpy=0.00000 0.0000 0.00000
- joint head_rzdammy: axis 1.00000 0.00000 0.00000 -> (none); origin xyz=0.00000 0.00000 0.00000 rpy=0.00000 -0.00000 0.00000 -> xyz=0.00000 0.00000 0.00000 rpy=0.00000 0.0000 0.00000
- joint left_ankle_rx: origin xyz=-0.01479 -0.42687 -0.03743 rpy=0.00000 -0.00000 0.00000 -> xyz=-0.01479 -0.42687 -0.03743 rpy=0.00000 0.0000 0.00000
- joint left_ankle_ry: origin xyz=0.00000 0.00000 0.00000 rpy=0.00000 -0.00000 0.00000 -> xyz=0.00000 0.00000 0.00000 rpy=0.00000 0.0000 0.00000
- joint left_ankle_rz: origin xyz=0.00000 0.00000 0.00000 rpy=0.00000 -0.00000 0.00000 -> xyz=0.00000 0.00000 0.00000 rpy=0.00000 0.0000 0.00000
- joint left_ankle_rzdammy: axis 0.00000 0.00000 0.00000 -> (none); origin xyz=0.00000 0.00000 0.00000 rpy=0.00000 -0.00000 0.00000 -> xyz=0.00000 0.00000 0.00000 rpy=0.00000 0.0000 0.00000
- joint left_clavicle_rx: origin xyz=0.07170 0.11400 -0.01890 rpy=0.00000 -0.00000 0.00000 -> xyz=0.07170 0.11400 -0.01890 rpy=0.00000 0.0000 0.00000
- joint left_clavicle_ry: origin xyz=0.00000 0.00000 0.00000 rpy=0.00000 -0.00000 0.00000 -> xyz=0.00000 0.00000 0.00000 rpy=0.00000 0.0000 0.00000
- joint left_clavicle_rz: origin xyz=0.00000 0.00000 0.00000 rpy=0.00000 -0.00000 0.00000 -> xyz=0.00000 0.00000 0.00000 rpy=0.00000 0.0000 0.00000
- joint left_clavicle_rzdammy: axis 0.00000 0.00000 0.00000 -> (none); origin xyz=0.00000 0.00000 0.00000 rpy=0.00000 -0.00000 0.00000 -> xyz=0.00000 0.00000 0.00000 rpy=0.00000 0.0000 0.00000
- joint left_elbow_rx: origin xyz=0.25533 -0.01565 -0.02295 rpy=0.00000 -0.00000 0.00000 -> xyz=0.25533 -0.01565 -0.02295 rpy=0.00000 0.0000 0.00000
- joint left_elbow_ry: origin xyz=0.00000 0.00000 0.00000 rpy=0.00000 -0.00000 0.00000 -> xyz=0.00000 0.00000 0.00000 rpy=0.00000 0.0000 0.00000
- joint left_elbow_rz: origin xyz=0.00000 0.00000 0.00000 rpy=0.00000 -0.00000 0.00000 -> xyz=0.00000 0.00000 0.00000 rpy=0.00000 0.0000 0.00000
- joint left_elbow_rzdammy: axis 0.00000 0.00000 0.00000 -> (none); origin xyz=0.00000 0.00000 0.00000 rpy=0.00000 -0.00000 0.00000 -> xyz=0.00000 0.00000 0.00000 rpy=0.00000 0.0000 0.00000
- joint left_foot_rx: origin xyz=0.04105 -0.06029 0.12204 rpy=0.00000 -0.00000 0.00000 -> xyz=0.04105 -0.06029 0.12204 rpy=0.00000 0.0000 0.00000
- joint left_foot_ry: origin xyz=0.00000 0.00000 0.00000 rpy=0.00000 -0.00000 0.00000 -> xyz=0.00000 0.00000 0.00000 rpy=0.00000 0.0000 0.00000
- joint left_foot_rz: origin xyz=0.00000 0.00000 0.00000 rpy=0.00000 -0.00000 0.00000 -> xyz=0.00000 0.00000 0.00000 rpy=0.00000 0.0000 0.00000
- joint left_foot_rzdammy: axis 0.00000 0.00000 0.00000 -> (none); origin xyz=0.00000 0.00000 0.00000 rpy=0.00000 -0.00000 0.00000 -> xyz=0.00000 0.00000 0.00000 rpy=0.00000 0.0000 0.00000
- joint left_hand_rx: origin xyz=0.08669 -0.01064 -0.01559 rpy=0.00000 -0.00000 0.00000 -> xyz=0.08669 -0.01064 -0.01559 rpy=0.00000 0.0000 0.00000
- joint left_hand_ry: origin xyz=0.00000 0.00000 0.00000 rpy=0.00000 -0.00000 0.00000 -> xyz=0.00000 0.00000 0.00000 rpy=0.00000 0.0000 0.00000
- joint left_hand_rz: origin xyz=0.00000 0.00000 0.00000 rpy=0.00000 -0.00000 0.00000 -> xyz=0.00000 0.00000 0.00000 rpy=0.00000 0.0000 0.00000
- joint left_hand_rzdammy: axis 1.00000 0.00000 0.00000 -> (none); limit lower=-2.50000 upper=2.50000 effort=1000.00000 velocity=0.50000 -> (none); origin xyz=0.00000 0.00000 0.00000 rpy=0.00000 -0.00000 0.00000 -> xyz=0.00000 0.00000 0.00000 rpy=0.00000 0.0000 0.00000; type revolute -> fixed
- joint left_heel: axis 0.00000 0.00000 0.00000 -> (none); origin xyz=0.00000 0.00000 0.00000 rpy=0.00000 -0.00000 0.00000 -> xyz=0.00000 0.00000 0.00000 rpy=0.00000 0.0000 0.00000
- joint left_hip_rx: origin xyz=0.05858 -0.08228 -0.01766 rpy=0.00000 -0.00000 0.00000 -> xyz=0.05858 -0.08228 -0.01766 rpy=0.00000 0.0000 0.00000
- joint left_hip_ry: origin xyz=0.00000 0.00000 0.00000 rpy=0.00000 -0.00000 0.00000 -> xyz=0.00000 0.00000 0.00000 rpy=0.00000 0.0000 0.00000
- joint left_hip_rz: origin xyz=0.00000 0.00000 0.00000 rpy=0.00000 -0.00000 0.00000 -> xyz=0.00000 0.00000 0.00000 rpy=0.00000 0.0000 0.00000
- joint left_hip_rzdammy: axis 0.00000 0.00000 0.00000 -> (none); origin xyz=0.00000 0.00000 0.00000 rpy=0.00000 -0.00000 0.00000 -> xyz=0.00000 0.00000 0.00000 rpy=0.00000 0.0000 0.00000
- joint left_knee_rx: origin xyz=0.04345 -0.38647 0.00804 rpy=0.00000 -0.00000 0.00000 -> xyz=0.04345 -0.38647 0.00804 rpy=0.00000 0.0000 0.00000
- joint left_knee_ry: origin xyz=0.00000 0.00000 0.00000 rpy=0.00000 -0.00000 0.00000 -> xyz=0.00000 0.00000 0.00000 rpy=0.00000 0.0000 0.00000
- joint left_knee_rz: origin xyz=0.00000 0.00000 0.00000 rpy=0.00000 -0.00000 0.00000 -> xyz=0.00000 0.00000 0.00000 rpy=0.00000 0.0000 0.00000
- joint left_knee_rzdammy: origin xyz=0.00000 0.00000 0.00000 rpy=0.00000 -0.00000 0.00000 -> xyz=0.00000 0.00000 0.00000 rpy=0.00000 0.0000 0.00000
- joint left_lowarm_rx: origin xyz=0.26571 0.01270 -0.00737 rpy=0.00000 -0.00000 0.00000 -> xyz=0.26571 0.01270 -0.00737 rpy=0.00000 0.0000 0.00000
- joint left_lowarm_ry: origin xyz=0.00000 0.00000 0.00000 rpy=0.00000 -0.00000 0.00000 -> xyz=0.00000 0.00000 0.00000 rpy=0.00000 0.0000 0.00000
- joint left_lowarm_rz: origin xyz=0.00000 0.00000 0.00000 rpy=0.00000 -0.00000 0.00000 -> xyz=0.00000 0.00000 0.00000 rpy=0.00000 0.0000 0.00000
- joint left_lowarm_rzdammy: axis 0.00000 0.00000 0.00000 -> (none); origin xyz=0.00000 0.00000 0.00000 rpy=0.00000 -0.00000 0.00000 -> xyz=0.00000 0.00000 0.00000 rpy=0.00000 0.0000 0.00000
- joint left_shoulder_rx: origin xyz=0.12292 0.04521 -0.01905 rpy=0.00000 -0.00000 0.00000 -> xyz=0.12292 0.04521 -0.01905 rpy=0.00000 0.0000 0.00000
- joint left_shoulder_ry: origin xyz=0.00000 0.00000 0.00000 rpy=0.00000 -0.00000 0.00000 -> xyz=0.00000 0.00000 0.00000 rpy=0.00000 0.0000 0.00000
- joint left_shoulder_rz: origin xyz=0.00000 0.00000 0.00000 rpy=0.00000 -0.00000 0.00000 -> xyz=0.00000 0.00000 0.00000 rpy=0.00000 0.0000 0.00000
- joint left_shoulder_rzdammy: axis 0.00000 0.00000 0.00000 -> (none); origin xyz=0.00000 0.00000 0.00000 rpy=0.00000 -0.00000 0.00000 -> xyz=0.00000 0.00000 0.00000 rpy=0.00000 0.0000 0.00000
- joint left_toe: axis 0.00000 0.00000 0.00000 -> (none); origin xyz=0.00000 0.00000 0.00000 rpy=1.57080 -0.00000 0.00000 -> xyz=0.00000 0.00000 0.00000 rpy=1.57080 0.0000 0.00000
- joint neck_rx: origin xyz=-0.01339 0.21164 -0.03347 rpy=0.00000 -0.00000 0.00000 -> xyz=-0.01339 0.21164 -0.03347 rpy=0.00000 0.0000 0.00000
- joint neck_ry: origin xyz=0.00000 0.00000 0.00000 rpy=0.00000 -0.00000 0.00000 -> xyz=0.00000 0.00000 0.00000 rpy=0.00000 0.0000 0.00000
- joint neck_rz: origin xyz=0.00000 0.00000 0.00000 rpy=0.00000 -0.00000 0.00000 -> xyz=0.00000 0.00000 0.00000 rpy=0.00000 0.0000 0.00000
- joint neck_rzdammy: axis 0.00000 0.00000 0.00000 -> (none); origin xyz=0.00000 0.00000 0.00000 rpy=0.00000 -0.00000 0.00000 -> xyz=0.00000 0.00000 0.00000 rpy=0.00000 0.0000 0.00000
- joint pelvis: origin xyz=0.00000 0.00000 0.00000 rpy=0.00000 -0.00000 0.00000 -> xyz=0.00000 0.00000 0.00000 rpy=0.00000 0.0000 0.00000
- joint right_ankle_rx: origin xyz=0.01906 -0.42005 -0.03456 rpy=0.00000 -0.00000 0.00000 -> xyz=0.01906 -0.42005 -0.03456 rpy=0.00000 0.0000 0.00000
- joint right_ankle_ry: origin xyz=0.00000 0.00000 0.00000 rpy=0.00000 -0.00000 0.00000 -> xyz=0.00000 0.00000 0.00000 rpy=0.00000 0.0000 0.00000
- joint right_ankle_rz: origin xyz=0.00000 0.00000 0.00000 rpy=0.00000 -0.00000 0.00000 -> xyz=0.00000 0.00000 0.00000 rpy=0.00000 0.0000 0.00000
- joint right_ankle_rzdammy: axis 0.00000 0.00000 0.00000 -> (none); origin xyz=0.00000 0.00000 0.00000 rpy=0.00000 -0.00000 0.00000 -> xyz=0.00000 0.00000 0.00000 rpy=0.00000 0.0000 0.00000
- joint right_clavicle_rx: origin xyz=-0.08295 0.11247 -0.02371 rpy=0.00000 -0.00000 0.00000 -> xyz=-0.08295 0.11247 -0.02371 rpy=0.00000 0.0000 0.00000
- joint right_clavicle_ry: origin xyz=0.00000 0.00000 0.00000 rpy=0.00000 -0.00000 0.00000 -> xyz=0.00000 0.00000 0.00000 rpy=0.00000 0.0000 0.00000
- joint right_clavicle_rz: origin xyz=0.00000 0.00000 0.00000 rpy=0.00000 -0.00000 0.00000 -> xyz=0.00000 0.00000 0.00000 rpy=0.00000 0.0000 0.00000
- joint right_clavicle_rzdammy: axis 0.00000 0.00000 0.00000 -> (none); origin xyz=0.00000 0.00000 0.00000 rpy=0.00000 -0.00000 0.00000 -> xyz=0.00000 0.00000 0.00000 rpy=0.00000 0.0000 0.00000
- joint right_elbow_rx: origin xyz=-0.26013 -0.01437 -0.03127 rpy=0.00000 -0.00000 0.00000 -> xyz=-0.26013 -0.01437 -0.03127 rpy=0.00000 0.0000 0.00000
- joint right_elbow_ry: origin xyz=0.00000 0.00000 0.00000 rpy=0.00000 -0.00000 0.00000 -> xyz=0.00000 0.00000 0.00000 rpy=0.00000 0.0000 0.00000
- joint right_elbow_rz: origin xyz=0.00000 0.00000 0.00000 rpy=0.00000 -0.00000 0.00000 -> xyz=0.00000 0.00000 0.00000 rpy=0.00000 0.0000 0.00000
- joint right_elbow_rzdammy: axis 0.00000 0.00000 0.00000 -> (none); origin xyz=0.00000 0.00000 0.00000 rpy=0.00000 -0.00000 0.00000 -> xyz=0.00000 0.00000 0.00000 rpy=0.00000 0.0000 0.00000
- joint right_foot_rx: origin xyz=-0.03484 -0.06211 0.13032 rpy=0.00000 -0.00000 0.00000 -> xyz=-0.03484 -0.06211 0.13032 rpy=0.00000 0.0000 0.00000
- joint right_foot_ry: origin xyz=0.00000 0.00000 0.00000 rpy=0.00000 -0.00000 0.00000 -> xyz=0.00000 0.00000 0.00000 rpy=0.00000 0.0000 0.00000
- joint right_foot_rz: origin xyz=0.00000 0.00000 0.00000 rpy=0.00000 -0.00000 0.00000 -> xyz=0.00000 0.00000 0.00000 rpy=0.00000 0.0000 0.00000
- joint right_foot_rzdammy: axis 0.00000 0.00000 0.00000 -> (none); origin xyz=0.00000 0.00000 0.00000 rpy=0.00000 -0.00000 0.00000 -> xyz=0.00000 0.00000 0.00000 rpy=0.00000 0.0000 0.00000
- joint right_hand_rx: origin xyz=-0.08875 -0.00865 -0.01011 rpy=0.00000 -0.00000 0.00000 -> xyz=-0.08875 -0.00865 -0.01011 rpy=0.00000 0.0000 0.00000
- joint right_hand_ry: origin xyz=0.00000 0.00000 0.00000 rpy=0.00000 -0.00000 0.00000 -> xyz=0.00000 0.00000 0.00000 rpy=0.00000 0.0000 0.00000
- joint right_hand_rz: origin xyz=0.00000 0.00000 0.00000 rpy=0.00000 -0.00000 0.00000 -> xyz=0.00000 0.00000 0.00000 rpy=0.00000 0.0000 0.00000
- joint right_hand_rzdammy: axis 1.00000 0.00000 0.00000 -> (none); limit lower=-2.50000 upper=2.50000 effort=1000.00000 velocity=0.50000 -> (none); origin xyz=0.00000 0.00000 0.00000 rpy=0.00000 -0.00000 0.00000 -> xyz=0.00000 0.00000 0.00000 rpy=0.00000 0.0000 0.00000; type revolute -> fixed
- joint right_heel: axis 0.00000 0.00000 0.00000 -> (none); origin xyz=0.00000 0.00000 0.00000 rpy=0.00000 -0.00000 0.00000 -> xyz=0.00000 0.00000 0.00000 rpy=0.00000 0.0000 0.00000
- joint right_hip_rx: origin xyz=-0.06031 -0.09051 -0.01354 rpy=0.00000 -0.00000 0.00000 -> xyz=-0.06031 -0.09051 -0.01354 rpy=0.00000 0.0000 0.00000
- joint right_hip_ry: origin xyz=0.00000 0.00000 0.00000 rpy=0.00000 -0.00000 0.00000 -> xyz=0.00000 0.00000 0.00000 rpy=0.00000 0.0000 0.00000
- joint right_hip_rz: origin xyz=0.00000 0.00000 0.00000 rpy=0.00000 -0.00000 0.00000 -> xyz=0.00000 0.00000 0.00000 rpy=0.00000 0.0000 0.00000
- joint right_hip_rzdammy: axis 0.00000 0.00000 0.00000 -> (none); origin xyz=0.00000 0.00000 0.00000 rpy=0.00000 -0.00000 0.00000 -> xyz=0.00000 0.00000 0.00000 rpy=0.00000 0.0000 0.00000
- joint right_knee_rx: origin xyz=-0.04326 -0.38369 -0.00484 rpy=0.00000 -0.00000 0.00000 -> xyz=-0.04326 -0.38369 -0.00484 rpy=0.00000 0.0000 0.00000
- joint right_knee_ry: origin xyz=0.00000 0.00000 0.00000 rpy=0.00000 -0.00000 0.00000 -> xyz=0.00000 0.00000 0.00000 rpy=0.00000 0.0000 0.00000
- joint right_knee_rz: origin xyz=0.00000 0.00000 0.00000 rpy=0.00000 -0.00000 0.00000 -> xyz=0.00000 0.00000 0.00000 rpy=0.00000 0.0000 0.00000
- joint right_knee_rzdammy: axis 0.00000 0.00000 0.00000 -> (none); origin xyz=0.00000 0.00000 0.00000 rpy=0.00000 -0.00000 0.00000 -> xyz=0.00000 0.00000 0.00000 rpy=0.00000 0.0000 0.00000
- joint right_lowarm_rx: origin xyz=-0.26911 0.00679 -0.00603 rpy=0.00000 -0.00000 0.00000 -> xyz=-0.26911 0.00679 -0.00603 rpy=0.00000 0.0000 0.00000
- joint right_lowarm_ry: origin xyz=0.00000 0.00000 0.00000 rpy=0.00000 -0.00000 0.00000 -> xyz=0.00000 0.00000 0.00000 rpy=0.00000 0.0000 0.00000
- joint right_lowarm_rz: origin xyz=0.00000 0.00000 0.00000 rpy=0.00000 -0.00000 0.00000 -> xyz=0.00000 0.00000 0.00000 rpy=0.00000 0.0000 0.00000
- joint right_lowarm_rzdammy: axis 0.00000 0.00000 0.00000 -> (none); origin xyz=0.00000 0.00000 0.00000 rpy=0.00000 -0.00000 0.00000 -> xyz=0.00000 0.00000 0.00000 rpy=0.00000 0.0000 0.00000
- joint right_shoulder_rx: origin xyz=-0.11323 0.04685 -0.00847 rpy=0.00000 -0.00000 0.00000 -> xyz=-0.11323 0.04685 -0.00847 rpy=0.00000 0.0000 0.00000
- joint right_shoulder_ry: origin xyz=0.00000 0.00000 0.00000 rpy=0.00000 -0.00000 0.00000 -> xyz=0.00000 0.00000 0.00000 rpy=0.00000 0.0000 0.00000
- joint right_shoulder_rz: origin xyz=0.00000 0.00000 0.00000 rpy=0.00000 -0.00000 0.00000 -> xyz=0.00000 0.00000 0.00000 rpy=0.00000 0.0000 0.00000
- joint right_shoulder_rzdammy: axis 0.00000 0.00000 0.00000 -> (none); origin xyz=0.00000 0.00000 0.00000 rpy=0.00000 -0.00000 0.00000 -> xyz=0.00000 0.00000 0.00000 rpy=0.00000 0.0000 0.00000
- joint right_toe: origin xyz=0.00000 0.00000 0.00000 rpy=1.57080 -0.00000 0.00000 -> xyz=0.00000 0.00000 0.00000 rpy=1.57080 0.0000 0.00000
- joint spine_2_rx: origin xyz=0.00444 0.12440 -0.03839 rpy=0.00000 -0.00000 0.00000 -> xyz=0.00444 0.12440 -0.03839 rpy=0.00000 0.0000 0.00000
- joint spine_2_ry: origin xyz=0.00000 0.00000 0.00000 rpy=0.00000 -0.00000 0.00000 -> xyz=0.00000 0.00000 0.00000 rpy=0.00000 0.0000 0.00000
- joint spine_2_rz: origin xyz=0.00000 0.00000 0.00000 rpy=0.00000 -0.00000 0.00000 -> xyz=0.00000 0.00000 0.00000 rpy=0.00000 0.0000 0.00000
- joint spine_2_rzdammy: axis 0.00000 0.00000 0.00000 -> (none); origin xyz=0.00000 0.00000 0.00000 rpy=0.00000 -0.00000 0.00000 -> xyz=0.00000 0.00000 0.00000 rpy=0.00000 0.0000 0.00000
- joint spine_3_rx: origin xyz=0.00449 0.13796 0.02682 rpy=0.00000 -0.00000 0.00000 -> xyz=0.00449 0.13796 0.02682 rpy=0.00000 0.0000 0.00000
- joint spine_3_ry: origin xyz=0.00000 0.00000 0.00000 rpy=0.00000 -0.00000 0.00000 -> xyz=0.00000 0.00000 0.00000 rpy=0.00000 0.0000 0.00000
- joint spine_3_rz: origin xyz=0.00000 0.00000 0.00000 rpy=0.00000 -0.00000 0.00000 -> xyz=0.00000 0.00000 0.00000 rpy=0.00000 0.0000 0.00000
- joint spine_3_rzdammy: axis 0.00000 0.00000 0.00000 -> (none); origin xyz=0.00000 0.00000 0.00000 rpy=0.00000 -0.00000 0.00000 -> xyz=0.00000 0.00000 0.00000 rpy=0.00000 0.0000 0.00000
- joint spine_4_rx: origin xyz=-0.00226 0.05603 0.00286 rpy=0.00000 -0.00000 0.00000 -> xyz=-0.00226 0.05603 0.00286 rpy=0.00000 0.0000 0.00000
- joint spine_4_ry: origin xyz=0.00000 0.00000 0.00000 rpy=0.00000 -0.00000 0.00000 -> xyz=0.00000 0.00000 0.00000 rpy=0.00000 0.0000 0.00000
- joint spine_4_rz: origin xyz=0.00000 0.00000 0.00000 rpy=0.00000 -0.00000 0.00000 -> xyz=0.00000 0.00000 0.00000 rpy=0.00000 0.0000 0.00000
- joint spine_4_rzdammy: axis 0.00000 0.00000 0.00000 -> (none); origin xyz=0.00000 0.00000 0.00000 rpy=0.00000 -0.00000 0.00000 -> xyz=0.00000 0.00000 0.00000 rpy=0.00000 0.0000 0.00000
