Commit message: remove all redundant radius and mass for fake links. fix self collision issue

File: ref_mesh.urdf (robot description, URDF)
Before this commit: robot human, 98 links, 97 joints
Links:
- link head_rx: mass 0.00001 -> 0.00000
- link head_ry: mass 0.00001 -> 0.00000
- link head_rz: mass 0.00001 -> 0.00000; geometry collision sphere radius=0.00000; visual sphere radius=0.00000
- link left_ankle_rx: mass 0.00001 -> 0.00000
- link left_ankle_ry: mass 0.00001 -> 0.00000
- link left_ankle_rz: mass 0.00001 -> 0.00000; geometry collision sphere radius=0.00000; visual sphere radius=0.00000
- link left_clavicle_rx: mass 0.00001 -> 0.00000
- link left_clavicle_ry: mass 0.00001 -> 0.00000
- link left_clavicle_rz: mass 0.00001 -> 0.00000; geometry collision sphere radius=0.00000; visual sphere radius=0.00000
- link left_elbow_rx: mass 0.00001 -> 0.00000; geometry collision sphere radius=0.00000; visual sphere radius=0.00000
- link left_elbow_ry: mass 0.00001 -> 0.00000
- link left_elbow_rz: mass 0.00001 -> 0.00000; geometry collision sphere radius=0.00000; visual sphere radius=0.00000
- link left_foot_rx: mass 0.00001 -> 0.00000
- link left_foot_ry: mass 0.00001 -> 0.00000
- link left_foot_rz: mass 0.00001 -> 0.00000; geometry collision sphere radius=0.00000; visual sphere radius=0.00000
- link left_hand_rx: mass 0.00001 -> 0.00000
- link left_hand_ry: mass 0.00001 -> 0.00000
- link left_hand_rz: mass 0.00001 -> 0.00000; geometry collision sphere radius=0.00000; visual sphere radius=0.00000
- link left_heel: mass 0.00001 -> 0.00000
- link left_knee_rx: mass 0.00001 -> 0.00000
- link left_knee_ry: mass 0.00001 -> 0.00000
- link left_knee_rz: mass 0.00001 -> 0.00000; geometry collision sphere radius=0.00000; visual sphere radius=0.00000
- link left_lowarm_rx: mass 0.00001 -> 0.00000
- link left_lowarm_ry: mass 0.00001 -> 0.00000
- link left_lowarm_rz: mass 0.00001 -> 0.00000; geometry collision sphere radius=0.00000; visual sphere radius=0.00000
- link left_shoulder_rx: mass 0.00001 -> 0.00000
- link left_shoulder_ry: mass 0.00001 -> 0.00000
- link left_shoulder_rz: mass 0.00001 -> 0.00000; geometry collision sphere radius=0.00000; visual sphere radius=0.00000
- link left_toe: mass 0.00001 -> 0.00000
- link neck_rx: mass 0.00001 -> 0.00000; geometry collision sphere radius=0.00000; visual sphere radius=0.00000
- link neck_ry: mass 0.00001 -> 0.00000
- link neck_rz: mass 0.00001 -> 0.00000
- link right_ankle_rx: mass 0.00001 -> 0.00000
- link right_ankle_ry: mass 0.00001 -> 0.00000
- link right_ankle_rz: mass 0.00001 -> 0.00000; geometry collision sphere radius=0.00000; visual sphere radius=0.00000
- link right_clavicle_rx: mass 0.00001 -> 0.00000
- link right_clavicle_ry: mass 0.00001 -> 0.00000
- link right_clavicle_rz: mass 0.00001 -> 0.00000; geometry collision sphere radius=0.00000; visual sphere radius=0.00000
- link right_elbow_rx: mass 0.00001 -> 0.00000; geometry collision sphere radius=0.00000; visual sphere radius=0.00000
- link right_elbow_ry: mass 0.00001 -> 0.00000
- link right_elbow_rz: mass 0.00001 -> 0.00000; geometry collision sphere radius=0.00000; visual sphere radius=0.00000
- link right_foot_rx: mass 0.00001 -> 0.00000
- link right_foot_ry: mass 0.00001 -> 0.00000
- link right_foot_rz: mass 0.00001 -> 0.00000; geometry collision sphere radius=0.00000; visual sphere radius=0.00000
- link right_hand_rx: mass 0.00001 -> 0.00000
- link right_hand_ry: mass 0.00001 -> 0.00000
- link right_hand_rz: mass 0.00001 -> 0.00000; geometry collision sphere radius=0.00000; visual sphere radius=0.00000
- link right_heel: mass 0.00001 -> 0.00000
- link right_hip_rx: mass 0.00001 -> 0.00000
- link right_hip_ry: mass 0.00001 -> 0.00000
- link right_hip_rz: mass 0.00001 -> 0.00000
- link right_knee_rx: mass 0.00001 -> 0.00000
- link right_knee_ry: mass 0.00001 -> 0.00000
- link right_knee_rz: mass 0.00001 -> 0.00000; geometry collision sphere radius=0.00000; visual sphere radius=0.00000
- link right_lowarm_rx: mass 0.00001 -> 0.00000
- link right_lowarm_ry: mass 0.00001 -> 0.00000
- link right_lowarm_rz: mass 0.00001 -> 0.00000; geometry collision sphere radius=0.00000; visual sphere radius=0.00000
- link right_shoulder_rx: mass 0.00001 -> 0.00000
- link right_shoulder_ry: mass 0.00001 -> 0.00000
- link right_shoulder_rz: mass 0.00001 -> 0.00000; geometry collision sphere radius=0.00000; visual sphere radius=0.00000
- link right_toe: mass 0.00001 -> 0.00000
- link spine_2_rx: mass 0.00001 -> 0.00000
- link spine_2_ry: mass 0.00001 -> 0.00000
- link spine_2_rz: mass 0.00001 -> 0.00000; geometry collision sphere radius=0.00000; visual sphere radius=0.00000
- link spine_3_rx: mass 0.00001 -> 0.00000
- link spine_3_ry: mass 0.00001 -> 0.00000
- link spine_3_rz: mass 0.00001 -> 0.00000; geometry collision sphere radius=0.00000; visual sphere radius=0.00000
- link spine_4_rx: mass 0.00001 -> 0.00000
- link spine_4_ry: mass 0.00001 -> 0.00000
- link spine_4_rz: mass 0.00001 -> 0.00000; geometry collision sphere radius=0.00000; visual sphere radius=0.00000
Joints:
- joint head_rx: limit lower=-2.50000 upper=2.50000 effort=1000.00000 velocity=0.50000 -> lower=-3.14 upper=3.14 effort=1000.00000 velocity=0.50000
- joint head_ry: limit lower=-2.50000 upper=2.50000 effort=1000.00000 velocity=0.50000 -> lower=-3.14 upper=3.14 effort=1000.00000 velocity=0.50000
- joint head_rz: limit lower=-2.50000 upper=2.50000 effort=1000.00000 velocity=0.50000 -> lower=-3.14 upper=3.14 effort=1000.00000 velocity=0.50000
- joint left_ankle_rx: limit lower=-0.40000 upper=0.70000 effort=1000.00000 velocity=0.50000 -> lower=-3.14 upper=3.14 effort=1000.00000 velocity=0.50000
- joint left_ankle_ry: limit lower=-0.50000 upper=0.50000 effort=1000.00000 velocity=0.50000 -> lower=-3.14 upper=3.14 effort=1000.00000 velocity=0.50000
- joint left_ankle_rz: limit lower=-0.40000 upper=0.40000 effort=1000.00000 velocity=0.50000 -> lower=-3.14 upper=3.14 effort=1000.00000 velocity=0.50000
- joint left_clavicle_rx: limit lower=-2.50000 upper=2.50000 effort=1000.00000 velocity=0.50000 -> lower=-3.14 upper=3.14 effort=1000.00000 velocity=0.50000
- joint left_clavicle_ry: limit lower=-0.60000 upper=0.40000 effort=1000.00000 velocity=0.50000 -> lower=-3.14 upper=3.14 effort=1000.00000 velocity=0.50000
- joint left_clavicle_rz: limit lower=-0.40000 upper=0.40000 effort=1000.00000 velocity=0.50000 -> lower=-3.14 upper=3.14 effort=1000.00000 velocity=0.50000
- joint left_elbow_rx: limit lower=-1.40000 upper=0.90000 effort=1000.00000 velocity=0.50000 -> lower=-3.14 upper=3.14 effort=1000.00000 velocity=0.50000
- joint left_elbow_ry: limit lower=-2.70000 upper=0.00000 effort=1000.00000 velocity=0.50000 -> lower=-3.14 upper=3.14 effort=1000.00000 velocity=0.50000
- joint left_elbow_rz: limit lower=-2.50000 upper=2.50000 effort=1000.00000 velocity=0.50000 -> lower=-3.14 upper=3.14 effort=1000.00000 velocity=0.50000
- joint left_foot_rx: limit lower=-2.50000 upper=2.50000 effort=1000.00000 velocity=0.50000 -> lower=-3.14 upper=3.14 effort=1000.00000 velocity=0.50000
- joint left_foot_ry: limit lower=-2.50000 upper=2.50000 effort=1000.00000 velocity=0.50000 -> lower=-3.14 upper=3.14 effort=1000.00000 velocity=0.50000
- joint left_foot_rz: limit lower=0.00000 upper=0.00000 effort=0.00000 velocity=0.00000 -> lower=-3.14 upper=3.14 effort=0.00000 velocity=0.00000
- joint left_hand_rx: limit lower=-2.50000 upper=2.50000 effort=1000.00000 velocity=0.50000 -> lower=-3.14 upper=3.14 effort=1000.00000 velocity=0.50000
- joint left_hand_ry: limit lower=-2.50000 upper=2.50000 effort=1000.00000 velocity=0.50000 -> lower=-3.14 upper=3.14 effort=1000.00000 velocity=0.50000
- joint left_hand_rz: limit lower=-2.50000 upper=2.50000 effort=1000.00000 velocity=0.50000 -> lower=-3.14 upper=3.14 effort=1000.00000 velocity=0.50000
- joint left_hip_rx: limit lower=-2.50000 upper=1.40000 effort=1000.00000 velocity=0.50000 -> lower=-3.14 upper=3.14 effort=1000.00000 velocity=0.50000
- joint left_hip_ry: limit lower=-0.60000 upper=0.60000 effort=1000.00000 velocity=0.50000 -> lower=-3.14 upper=3.14 effort=1000.00000 velocity=0.50000
- joint left_hip_rz: limit lower=-0.80000 upper=1.40000 effort=1000.00000 velocity=0.50000 -> lower=-3.14 upper=3.14 effort=1000.00000 velocity=0.50000
- joint left_knee_rx: limit lower=-0.10000 upper=2.50000 effort=1000.00000 velocity=0.50000 -> lower=-3.14 upper=3.14 effort=1000.00000 velocity=0.50000
- joint left_knee_ry: limit lower=-2.50000 upper=2.50000 effort=1000.00000 velocity=0.50000 -> lower=-3.14 upper=3.14 effort=1000.00000 velocity=0.50000
- joint left_knee_rz: limit lower=-2.50000 upper=2.50000 effort=1000.00000 velocity=0.50000 -> lower=-3.14 upper=3.14 effort=1000.00000 velocity=0.50000
- joint left_lowarm_rx: limit lower=-2.50000 upper=2.50000 effort=1000.00000 velocity=0.50000 -> lower=-3.14 upper=3.14 effort=1000.00000 velocity=0.50000
- joint left_lowarm_ry: limit lower=-2.50000 upper=2.50000 effort=1000.00000 velocity=0.50000 -> lower=-3.14 upper=3.14 effort=1000.00000 velocity=0.50000
- joint left_lowarm_rz: limit lower=-2.50000 upper=2.50000 effort=1000.00000 velocity=0.50000 -> lower=-3.14 upper=3.14 effort=1000.00000 velocity=0.50000
- joint left_shoulder_rx: limit lower=-2.50000 upper=2.50000 effort=1000.00000 velocity=0.50000 -> lower=-3.14 upper=3.14 effort=1000.00000 velocity=0.50000
- joint left_shoulder_ry: limit lower=-2.00000 upper=0.60000 effort=1000.00000 velocity=0.50000 -> lower=-3.14 upper=3.14 effort=1000.00000 velocity=0.50000
- joint left_shoulder_rz: limit lower=-1.00000 upper=1.00000 effort=1000.00000 velocity=0.50000 -> lower=-3.14 upper=3.14 effort=1000.00000 velocity=0.50000
- joint neck_rx: limit lower=-0.60000 upper=0.60000 effort=1000.00000 velocity=0.50000 -> lower=-3.14 upper=3.14 effort=1000.00000 velocity=0.50000
- joint neck_ry: limit lower=-0.60000 upper=0.60000 effort=1000.00000 velocity=0.50000 -> lower=-3.14 upper=3.14 effort=1000.00000 velocity=0.50000
- joint neck_rz: limit lower=-0.30000 upper=0.30000 effort=1000.00000 velocity=0.50000 -> lower=-3.14 upper=3.14 effort=1000.00000 velocity=0.50000
- joint right_ankle_rx: limit lower=-0.40000 upper=0.70000 effort=1000.00000 velocity=0.50000 -> lower=-3.14 upper=3.14 effort=1000.00000 velocity=0.50000
- joint right_ankle_ry: limit lower=-0.50000 upper=0.50000 effort=1000.00000 velocity=0.50000 -> lower=-3.14 upper=3.14 effort=1000.00000 velocity=0.50000
- joint right_ankle_rz: limit lower=-0.40000 upper=0.40000 effort=1000.00000 velocity=0.50000 -> lower=-3.14 upper=3.14 effort=1000.00000 velocity=0.50000
- joint right_clavicle_rx: limit lower=-2.50000 upper=2.50000 effort=1000.00000 velocity=0.50000 -> lower=-3.14 upper=3.14 effort=1000.00000 velocity=0.50000
- joint right_clavicle_ry: limit lower=-0.40000 upper=0.60000 effort=1000.00000 velocity=0.50000 -> lower=-3.14 upper=3.14 effort=1000.00000 velocity=0.50000
- joint right_clavicle_rz: limit lower=-0.40000 upper=0.40000 effort=1000.00000 velocity=0.50000 -> lower=-3.14 upper=3.14 effort=1000.00000 velocity=0.50000
- joint right_elbow_rx: limit lower=-1.40000 upper=0.90000 effort=1000.00000 velocity=0.50000 -> lower=-3.14 upper=3.14 effort=1000.00000 velocity=0.50000
- joint right_elbow_ry: limit lower=0.00000 upper=2.70000 effort=1000.00000 velocity=0.50000 -> lower=-3.14 upper=3.14 effort=1000.00000 velocity=0.50000
- joint right_elbow_rz: limit lower=-2.50000 upper=2.50000 effort=1000.00000 velocity=0.50000 -> lower=-3.14 upper=3.14 effort=1000.00000 velocity=0.50000
- joint right_foot_rx: limit lower=-2.50000 upper=2.50000 effort=1000.00000 velocity=0.50000 -> lower=-3.14 upper=3.14 effort=1000.00000 velocity=0.50000
- joint right_foot_ry: limit lower=-2.50000 upper=2.50000 effort=1000.00000 velocity=0.50000 -> lower=-3.14 upper=3.14 effort=1000.00000 velocity=0.50000
- joint right_foot_rz: limit lower=0.00000 upper=0.00000 effort=1000.00000 velocity=0.50000 -> lower=-3.14 upper=3.14 effort=1000.00000 velocity=0.50000
- joint right_hand_rx: limit lower=-2.50000 upper=2.50000 effort=1000.00000 velocity=0.50000 -> lower=-3.14 upper=3.14 effort=1000.00000 velocity=0.50000
- joint right_hand_ry: limit lower=-2.50000 upper=2.50000 effort=1000.00000 velocity=0.50000 -> lower=-3.14 upper=3.14 effort=1000.00000 velocity=0.50000
- joint right_hand_rz: limit lower=-2.50000 upper=2.50000 effort=1000.00000 velocity=0.50000 -> lower=-3.14 upper=3.14 effort=1000.00000 velocity=0.50000
- joint right_hip_rx: limit lower=-2.50000 upper=1.40000 effort=1000.00000 velocity=0.50000 -> lower=-3.14 upper=3.14 effort=1000.00000 velocity=0.50000
- joint right_hip_ry: limit lower=-0.60000 upper=0.60000 effort=1000.00000 velocity=0.50000 -> lower=-3.14 upper=3.14 effort=1000.00000 velocity=0.50000
- joint right_hip_rz: limit lower=-1.40000 upper=0.80000 effort=1000.00000 velocity=0.50000 -> lower=-3.14 upper=3.14 effort=1000.00000 velocity=0.50000
- joint right_knee_rx: limit lower=-0.10000 upper=2.50000 effort=1000.00000 velocity=0.50000 -> lower=-3.14 upper=3.14 effort=1000.00000 velocity=0.50000
- joint right_knee_ry: limit lower=-2.50000 upper=2.50000 effort=1000.00000 velocity=0.50000 -> lower=-3.14 upper=3.14 effort=1000.00000 velocity=0.50000
- joint right_knee_rz: limit lower=-2.50000 upper=2.50000 effort=1000.00000 velocity=0.50000 -> lower=-3.14 upper=3.14 effort=1000.00000 velocity=0.50000
- joint right_lowarm_rx: limit lower=-2.50000 upper=2.50000 effort=1000.00000 velocity=0.50000 -> lower=-3.14 upper=3.14 effort=1000.00000 velocity=0.50000
- joint right_lowarm_ry: limit lower=-2.50000 upper=2.50000 effort=1000.00000 velocity=0.50000 -> lower=-3.14 upper=3.14 effort=1000.00000 velocity=0.50000
- joint right_lowarm_rz: limit lower=-2.50000 upper=2.50000 effort=1000.00000 velocity=0.50000 -> lower=-3.14 upper=3.14 effort=1000.00000 velocity=0.50000
- joint right_shoulder_rx: limit lower=-2.50000 upper=2.50000 effort=1000.00000 velocity=0.50000 -> lower=-3.14 upper=3.14 effort=1000.00000 velocity=0.50000
- joint right_shoulder_ry: limit lower=-0.60000 upper=2.00000 effort=1000.00000 velocity=0.50000 -> lower=-3.14 upper=3.14 effort=1000.00000 velocity=0.50000
- joint right_shoulder_rz: limit lower=-1.00000 upper=1.00000 effort=1000.00000 velocity=0.50000 -> lower=-3.14 upper=3.14 effort=1000.00000 velocity=0.50000
- joint spine_2_rx: limit lower=-2.50000 upper=2.50000 effort=1000.00000 velocity=0.50000 -> lower=-3.14 upper=3.14 effort=1000.00000 velocity=0.50000
- joint spine_2_ry: limit lower=-2.50000 upper=2.50000 effort=1000.00000 velocity=0.50000 -> lower=-3.14 upper=3.14 effort=1000.00000 velocity=0.50000
- joint spine_2_rz: limit lower=-2.50000 upper=2.50000 effort=1000.00000 velocity=0.50000 -> lower=-3.14 upper=3.14 effort=1000.00000 velocity=0.50000
- joint spine_3_rx: limit lower=-2.50000 upper=2.50000 effort=1000.00000 velocity=0.50000 -> lower=-3.14 upper=3.14 effort=1000.00000 velocity=0.50000
- joint spine_3_ry: limit lower=-2.50000 upper=2.50000 effort=1000.00000 velocity=0.50000 -> lower=-3.14 upper=3.14 effort=1000.00000 velocity=0.50000
- joint spine_3_rz: limit lower=-2.50000 upper=2.50000 effort=1000.00000 velocity=0.50000 -> lower=-3.14 upper=3.14 effort=1000.00000 velocity=0.50000
- joint spine_4_rx: limit lower=-2.50000 upper=2.50000 effort=1000.00000 velocity=0.50000 -> lower=-3.14 upper=3.14 effort=1000.00000 velocity=0.50000
- joint spine_4_ry: limit lower=-2.50000 upper=2.50000 effort=1000.00000 velocity=0.50000 -> lower=-3.14 upper=3.14 effort=1000.00000 velocity=0.50000
- joint spine_4_rz: limit lower=-2.50000 upper=2.50000 effort=1000.00000 velocity=0.50000 -> lower=-3.14 upper=3.14 effort=1000.00000 velocity=0.50000
