Commit message: further fix self-collision and human fly away issue. code clean up

File: ref_mesh.urdf (robot description, URDF)
Before this commit: robot human, 98 links, 97 joints
Joints:
- joint head_rx: limit lower=-3.14 upper=3.14 effort=1000.00000 velocity=0.50000 -> lower=-3.14 upper=3.14 effort=1000.00000 velocity=0.00000
- joint head_ry: limit lower=-3.14 upper=3.14 effort=1000.00000 velocity=0.50000 -> lower=-3.14 upper=3.14 effort=1000.00000 velocity=0.00000
- joint head_rz: limit lower=-3.14 upper=3.14 effort=1000.00000 velocity=0.50000 -> lower=-3.14 upper=3.14 effort=1000.00000 velocity=0.00000
- joint left_ankle_rx: limit lower=-3.14 upper=3.14 effort=1000.00000 velocity=0.50000 -> lower=-3.14 upper=3.14 effort=1000.00000 velocity=0.00000
- joint left_ankle_ry: limit lower=-3.14 upper=3.14 effort=1000.00000 velocity=0.50000 -> lower=-3.14 upper=3.14 effort=1000.00000 velocity=0.00000
- joint left_ankle_rz: limit lower=-3.14 upper=3.14 effort=1000.00000 velocity=0.50000 -> lower=-3.14 upper=3.14 effort=1000.00000 velocity=0.00000
- joint left_clavicle_rx: limit lower=-3.14 upper=3.14 effort=1000.00000 velocity=0.50000 -> lower=-3.14 upper=3.14 effort=1000.00000 velocity=0.00000
- joint left_clavicle_ry: limit lower=-3.14 upper=3.14 effort=1000.00000 velocity=0.50000 -> lower=-3.14 upper=3.14 effort=1000.00000 velocity=0.00000
- joint left_clavicle_rz: limit lower=-3.14 upper=3.14 effort=1000.00000 velocity=0.50000 -> lower=-3.14 upper=3.14 effort=1000.00000 velocity=0.00000
- joint left_elbow_rx: limit lower=-3.14 upper=3.14 effort=1000.00000 velocity=0.50000 -> lower=-3.14 upper=3.14 effort=1000.00000 velocity=0.00000
- joint left_elbow_ry: limit lower=-3.14 upper=3.14 effort=1000.00000 velocity=0.50000 -> lower=-3.14 upper=3.14 effort=1000.00000 velocity=0.00000
- joint left_elbow_rz: limit lower=-3.14 upper=3.14 effort=1000.00000 velocity=0.50000 -> lower=-3.14 upper=3.14 effort=1000.00000 velocity=0.00000
- joint left_foot_rx: limit lower=-3.14 upper=3.14 effort=1000.00000 velocity=0.50000 -> lower=-3.14 upper=3.14 effort=1000.00000 velocity=0.00000
- joint left_foot_ry: limit lower=-3.14 upper=3.14 effort=1000.00000 velocity=0.50000 -> lower=-3.14 upper=3.14 effort=1000.00000 velocity=0.00000
- joint left_hand_rx: limit lower=-3.14 upper=3.14 effort=1000.00000 velocity=0.50000 -> lower=-3.14 upper=3.14 effort=1000.00000 velocity=0.00000
- joint left_hand_ry: limit lower=-3.14 upper=3.14 effort=1000.00000 velocity=0.50000 -> lower=-3.14 upper=3.14 effort=1000.00000 velocity=0.00000
- joint left_hand_rz: limit lower=-3.14 upper=3.14 effort=1000.00000 velocity=0.50000 -> lower=-3.14 upper=3.14 effort=1000.00000 velocity=0.00000
- joint left_hip_rx: limit lower=-3.14 upper=3.14 effort=1000.00000 velocity=0.50000 -> lower=-3.14 upper=3.14 effort=1000.00000 velocity=0.00000
- joint left_hip_ry: limit lower=-3.14 upper=3.14 effort=1000.00000 velocity=0.50000 -> lower=-3.14 upper=3.14 effort=1000.00000 velocity=0.00000
- joint left_hip_rz: limit lower=-3.14 upper=3.14 effort=1000.00000 velocity=0.50000 -> lower=-3.14 upper=3.14 effort=1000.00000 velocity=0.00000
- joint left_knee_rx: limit lower=-3.14 upper=3.14 effort=1000.00000 velocity=0.50000 -> lower=-3.14 upper=3.14 effort=1000.00000 velocity=0.00000
- joint left_knee_ry: limit lower=-3.14 upper=3.14 effort=1000.00000 velocity=0.50000 -> lower=-3.14 upper=3.14 effort=1000.00000 velocity=0.00000
- joint left_knee_rz: limit lower=-3.14 upper=3.14 effort=1000.00000 velocity=0.50000 -> lower=-3.14 upper=3.14 effort=1000.00000 velocity=0.00000
- joint left_lowarm_rx: limit lower=-3.14 upper=3.14 effort=1000.00000 velocity=0.50000 -> lower=-3.14 upper=3.14 effort=1000.00000 velocity=0.00000
- joint left_lowarm_ry: limit lower=-3.14 upper=3.14 effort=1000.00000 velocity=0.50000 -> lower=-3.14 upper=3.14 effort=1000.00000 velocity=0.00000
- joint left_lowarm_rz: limit lower=-3.14 upper=3.14 effort=1000.00000 velocity=0.50000 -> lower=-3.14 upper=3.14 effort=1000.00000 velocity=0.00000
- joint left_shoulder_rx: limit lower=-3.14 upper=3.14 effort=1000.00000 velocity=0.50000 -> lower=-3.14 upper=3.14 effort=1000.00000 velocity=0.00000
- joint left_shoulder_ry: limit lower=-3.14 upper=3.14 effort=1000.00000 velocity=0.50000 -> lower=-3.14 upper=3.14 effort=1000.00000 velocity=0.00000
- joint left_shoulder_rz: limit lower=-3.14 upper=3.14 effort=1000.00000 velocity=0.50000 -> lower=-3.14 upper=3.14 effort=1000.00000 velocity=0.00000
- joint neck_rx: limit lower=-3.14 upper=3.14 effort=1000.00000 velocity=0.50000 -> lower=-3.14 upper=3.14 effort=1000.00000 velocity=0.00000
- joint neck_ry: limit lower=-3.14 upper=3.14 effort=1000.00000 velocity=0.50000 -> lower=-3.14 upper=3.14 effort=1000.00000 velocity=0.00000
- joint neck_rz: limit lower=-3.14 upper=3.14 effort=1000.00000 velocity=0.50000 -> lower=-3.14 upper=3.14 effort=1000.00000 velocity=0.00000
- joint right_ankle_rx: limit lower=-3.14 upper=3.14 effort=1000.00000 velocity=0.50000 -> lower=-3.14 upper=3.14 effort=1000.00000 velocity=0.00000
- joint right_ankle_ry: limit lower=-3.14 upper=3.14 effort=1000.00000 velocity=0.50000 -> lower=-3.14 upper=3.14 effort=1000.00000 velocity=0.00000
- joint right_ankle_rz: limit lower=-3.14 upper=3.14 effort=1000.00000 velocity=0.50000 -> lower=-3.14 upper=3.14 effort=1000.00000 velocity=0.00000
- joint right_clavicle_rx: limit lower=-3.14 upper=3.14 effort=1000.00000 velocity=0.50000 -> lower=-3.14 upper=3.14 effort=1000.00000 velocity=0.00000
- joint right_clavicle_ry: limit lower=-3.14 upper=3.14 effort=1000.00000 velocity=0.50000 -> lower=-3.14 upper=3.14 effort=1000.00000 velocity=0.00000
- joint right_clavicle_rz: limit lower=-3.14 upper=3.14 effort=1000.00000 velocity=0.50000 -> lower=-3.14 upper=3.14 effort=1000.00000 velocity=0.00000
- joint right_elbow_rx: limit lower=-3.14 upper=3.14 effort=1000.00000 velocity=0.50000 -> lower=-3.14 upper=3.14 effort=1000.00000 velocity=0.00000
- joint right_elbow_ry: limit lower=-3.14 upper=3.14 effort=1000.00000 velocity=0.50000 -> lower=-3.14 upper=3.14 effort=1000.00000 velocity=0.00000
- joint right_elbow_rz: limit lower=-3.14 upper=3.14 effort=1000.00000 velocity=0.50000 -> lower=-3.14 upper=3.14 effort=1000.00000 velocity=0.00000
- joint right_foot_rx: limit lower=-3.14 upper=3.14 effort=1000.00000 velocity=0.50000 -> lower=-3.14 upper=3.14 effort=1000.00000 velocity=0.00000
- joint right_foot_ry: limit lower=-3.14 upper=3.14 effort=1000.00000 velocity=0.50000 -> lower=-3.14 upper=3.14 effort=1000.00000 velocity=0.00000
- joint right_foot_rz: limit lower=-3.14 upper=3.14 effort=1000.00000 velocity=0.50000 -> lower=-3.14 upper=3.14 effort=1000.00000 velocity=0.00000
- joint right_hand_rx: limit lower=-3.14 upper=3.14 effort=1000.00000 velocity=0.50000 -> lower=-3.14 upper=3.14 effort=1000.00000 velocity=0.00000
- joint right_hand_ry: limit lower=-3.14 upper=3.14 effort=1000.00000 velocity=0.50000 -> lower=-3.14 upper=3.14 effort=1000.00000 velocity=0.00000
- joint right_hand_rz: limit lower=-3.14 upper=3.14 effort=1000.00000 velocity=0.50000 -> lower=-3.14 upper=3.14 effort=1000.00000 velocity=0.00000
- joint right_hip_rx: limit lower=-3.14 upper=3.14 effort=1000.00000 velocity=0.50000 -> lower=-3.14 upper=3.14 effort=1000.00000 velocity=0.00000
- joint right_hip_ry: limit lower=-3.14 upper=3.14 effort=1000.00000 velocity=0.50000 -> lower=-3.14 upper=3.14 effort=1000.00000 velocity=0.00000
- joint right_hip_rz: limit lower=-3.14 upper=3.14 effort=1000.00000 velocity=0.50000 -> lower=-3.14 upper=3.14 effort=1000.00000 velocity=0.00000
- joint right_knee_rx: limit lower=-3.14 upper=3.14 effort=1000.00000 velocity=0.50000 -> lower=-3.14 upper=3.14 effort=1000.00000 velocity=0.00000
- joint right_knee_ry: limit lower=-3.14 upper=3.14 effort=1000.00000 velocity=0.50000 -> lower=-3.14 upper=3.14 effort=1000.00000 velocity=0.00000
- joint right_knee_rz: limit lower=-3.14 upper=3.14 effort=1000.00000 velocity=0.50000 -> lower=-3.14 upper=3.14 effort=1000.00000 velocity=0.00000
- joint right_lowarm_rx: limit lower=-3.14 upper=3.14 effort=1000.00000 velocity=0.50000 -> lower=-3.14 upper=3.14 effort=1000.00000 velocity=0.00000
- joint right_lowarm_ry: limit lower=-3.14 upper=3.14 effort=1000.00000 velocity=0.50000 -> lower=-3.14 upper=3.14 effort=1000.00000 velocity=0.00000
- joint right_lowarm_rz: limit lower=-3.14 upper=3.14 effort=1000.00000 velocity=0.50000 -> lower=-3.14 upper=3.14 effort=1000.00000 velocity=0.00000
- joint right_shoulder_rx: limit lower=-3.14 upper=3.14 effort=1000.00000 velocity=0.50000 -> lower=-3.14 upper=3.14 effort=1000.00000 velocity=0.00000
- joint right_shoulder_ry: limit lower=-3.14 upper=3.14 effort=1000.00000 velocity=0.50000 -> lower=-3.14 upper=3.14 effort=1000.00000 velocity=0.00000
- joint right_shoulder_rz: limit lower=-3.14 upper=3.14 effort=1000.00000 velocity=0.50000 -> lower=-3.14 upper=3.14 effort=1000.00000 velocity=0.00000
- joint spine_2_rx: limit lower=-3.14 upper=3.14 effort=1000.00000 velocity=0.50000 -> lower=-3.14 upper=3.14 effort=1000.00000 velocity=0.00000
- joint spine_2_ry: limit lower=-3.14 upper=3.14 effort=1000.00000 velocity=0.50000 -> lower=-3.14 upper=3.14 effort=1000.00000 velocity=0.00000
- joint spine_2_rz: limit lower=-3.14 upper=3.14 effort=1000.00000 velocity=0.50000 -> lower=-3.14 upper=3.14 effort=1000.00000 velocity=0.00000
- joint spine_3_rx: limit lower=-3.14 upper=3.14 effort=1000.00000 velocity=0.50000 -> lower=-3.14 upper=3.14 effort=1000.00000 velocity=0.00000
- joint spine_3_ry: limit lower=-3.14 upper=3.14 effort=1000.00000 velocity=0.50000 -> lower=-3.14 upper=3.14 effort=1000.00000 velocity=0.00000
- joint spine_3_rz: limit lower=-3.14 upper=3.14 effort=1000.00000 velocity=0.50000 -> lower=-3.14 upper=3.14 effort=1000.00000 velocity=0.00000
- joint spine_4_rx: limit lower=-3.14 upper=3.14 effort=1000.00000 velocity=0.50000 -> lower=-3.14 upper=3.14 effort=1000.00000 velocity=0.00000
- joint spine_4_ry: limit lower=-3.14 upper=3.14 effort=1000.00000 velocity=0.50000 -> lower=-3.14 upper=3.14 effort=1000.00000 velocity=0.00000
- joint spine_4_rz: limit lower=-3.14 upper=3.14 effort=1000.00000 velocity=0.50000 -> lower=-3.14 upper=3.14 effort=1000.00000 velocity=0.00000

Commit message: update axis rot for joint in urdf

File: ref_mesh.urdf (robot description, URDF)
Before this commit: robot human, 98 links, 97 joints
Links:
- removed link left_heel
- removed link left_toe
- removed link right_heel
- removed link right_toe
Joints:
- removed joint left_heel
- removed joint left_toe
- removed joint right_heel
- removed joint right_toe
- joint head_rx: axis 0.00000 1.00000 0.00000 -> 1.00000 0.00000 0.00000
- joint head_ry: axis 0.00000 0.00000 1.00000 -> 0.00000 1.00000 0.00000
- joint head_rz: axis 1.00000 0.00000 0.00000 -> 0.00000 0.00000 1.00000
- joint left_ankle_rx: axis 0.00000 1.00000 0.00000 -> 1.00000 0.00000 0.00000
- joint left_ankle_ry: axis 0.00000 0.00000 1.00000 -> 0.00000 1.00000 0.00000
- joint left_ankle_rz: axis 1.00000 0.00000 0.00000 -> 0.00000 0.00000 1.00000
- joint left_clavicle_rx: axis 0.00000 1.00000 0.00000 -> 1.00000 0.00000 0.00000
- joint left_clavicle_ry: axis 0.00000 0.00000 1.00000 -> 0.00000 1.00000 0.00000
- joint left_clavicle_rz: axis 1.00000 0.00000 0.00000 -> 0.00000 0.00000 1.00000
- joint left_elbow_rx: axis 0.00000 1.00000 0.00000 -> 1.00000 0.00000 0.00000
- joint left_elbow_ry: axis 0.00000 0.00000 1.00000 -> 0.00000 1.00000 0.00000
- joint left_elbow_rz: axis 1.00000 0.00000 0.00000 -> 0.00000 0.00000 1.00000
- joint left_foot_rx: axis 0.00000 1.00000 0.00000 -> 1.00000 0.00000 0.00000
- joint left_foot_ry: axis 0.00000 0.00000 1.00000 -> 0.00000 1.00000 0.00000
- joint left_foot_rz: axis 1.00000 0.00000 0.00000 -> 0.00000 0.00000 1.00000
- joint left_hand_rx: axis 0.00000 1.00000 0.00000 -> 1.00000 0.00000 0.00000
- joint left_hand_ry: axis 0.00000 0.00000 1.00000 -> 0.00000 1.00000 0.00000
- joint left_hand_rz: axis 1.00000 0.00000 0.00000 -> 0.00000 0.00000 1.00000
- joint left_hip_rx: axis 0.00000 1.00000 0.00000 -> 1.00000 0.00000 0.00000
- joint left_hip_ry: axis 0.00000 0.00000 1.00000 -> 0.00000 1.00000 0.00000
- joint left_hip_rz: axis 1.00000 0.00000 0.00000 -> 0.00000 0.00000 1.00000
- joint left_knee_rx: axis 0.00000 1.00000 0.00000 -> 1.00000 0.00000 0.00000
- joint left_knee_ry: axis 0.00000 0.00000 1.00000 -> 0.00000 1.00000 0.00000
- joint left_knee_rz: axis 1.00000 0.00000 0.00000 -> 0.00000 0.00000 1.00000
- joint left_lowarm_rx: axis 0.00000 1.00000 0.00000 -> 1.00000 0.00000 0.00000
- joint left_lowarm_ry: axis 0.00000 0.00000 1.00000 -> 0.00000 1.00000 0.00000
- joint left_lowarm_rz: axis 1.00000 0.00000 0.00000 -> 0.00000 0.00000 1.00000
- joint left_shoulder_rx: axis 0.00000 1.00000 0.00000 -> 1.00000 0.00000 0.00000
- joint left_shoulder_ry: axis 0.00000 0.00000 1.00000 -> 0.00000 1.00000 0.00000
- joint left_shoulder_rz: axis 1.00000 0.00000 0.00000 -> 0.00000 0.00000 1.00000
- joint neck_rx: axis 0.00000 1.00000 0.00000 -> 1.00000 0.00000 0.00000
- joint neck_ry: axis 0.00000 0.00000 1.00000 -> 0.00000 1.00000 0.00000
- joint neck_rz: axis 1.00000 0.00000 0.00000 -> 0.00000 0.00000 1.00000
- joint right_ankle_rx: axis 0.00000 1.00000 0.00000 -> 1.00000 0.00000 0.00000
- joint right_ankle_ry: axis 0.00000 0.00000 1.00000 -> 0.00000 1.00000 0.00000
- joint right_ankle_rz: axis 1.00000 0.00000 0.00000 -> 0.00000 0.00000 1.00000
- joint right_clavicle_rx: axis 0.00000 1.00000 0.00000 -> 1.00000 0.00000 0.00000
- joint right_clavicle_ry: axis 0.00000 0.00000 1.00000 -> 0.00000 1.00000 0.00000
- joint right_clavicle_rz: axis 1.00000 0.00000 0.00000 -> 0.00000 0.00000 1.00000
- joint right_elbow_rx: axis 0.00000 1.00000 0.00000 -> 1.00000 0.00000 0.00000
- joint right_elbow_ry: axis 0.00000 0.00000 1.00000 -> 0.00000 1.00000 0.00000
- joint right_elbow_rz: axis 1.00000 0.00000 0.00000 -> 0.00000 0.00000 1.00000
- joint right_foot_rx: axis 0.00000 1.00000 0.00000 -> 1.00000 0.00000 0.00000
- joint right_foot_ry: axis 0.00000 0.00000 1.00000 -> 0.00000 1.00000 0.00000
- joint right_foot_rz: axis 1.00000 0.00000 0.00000 -> 0.00000 0.00000 1.00000
- joint right_hand_rx: axis 0.00000 1.00000 0.00000 -> 1.00000 0.00000 0.00000
- joint right_hand_ry: axis 0.00000 0.00000 1.00000 -> 0.00000 1.00000 0.00000
- joint right_hand_rz: axis 1.00000 0.00000 0.00000 -> 0.00000 0.00000 1.00000
- joint right_hip_rx: axis 0.00000 1.00000 0.00000 -> 1.00000 0.00000 0.00000
- joint right_hip_ry: axis 0.00000 0.00000 1.00000 -> 0.00000 1.00000 0.00000
- joint right_hip_rz: axis 1.00000 0.00000 0.00000 -> 0.00000 0.00000 1.00000
- joint right_knee_rx: axis 0.00000 1.00000 0.00000 -> 1.00000 0.00000 0.00000
- joint right_knee_ry: axis 0.00000 0.00000 1.00000 -> 0.00000 1.00000 0.00000
- joint right_knee_rz: axis 1.00000 0.00000 0.00000 -> 0.00000 0.00000 1.00000
- joint right_lowarm_rx: axis 0.00000 1.00000 0.00000 -> 1.00000 0.00000 0.00000
- joint right_lowarm_ry: axis 0.00000 0.00000 1.00000 -> 0.00000 1.00000 0.00000
- joint right_lowarm_rz: axis 1.00000 0.00000 0.00000 -> 0.00000 0.00000 1.00000
- joint right_shoulder_rx: axis 0.00000 1.00000 0.00000 -> 1.00000 0.00000 0.00000
- joint right_shoulder_ry: axis 0.00000 0.00000 1.00000 -> 0.00000 1.00000 0.00000
- joint right_shoulder_rz: axis 1.00000 0.00000 0.00000 -> 0.00000 0.00000 1.00000
- joint spine_2_rx: axis 0.00000 1.00000 0.00000 -> 1.00000 0.00000 0.00000
- joint spine_2_ry: axis 0.00000 0.00000 1.00000 -> 0.00000 1.00000 0.00000
- joint spine_2_rz: axis 1.00000 0.00000 0.00000 -> 0.00000 0.00000 1.00000
- joint spine_3_rx: axis 0.00000 1.00000 0.00000 -> 1.00000 0.00000 0.00000
- joint spine_3_ry: axis 0.00000 0.00000 1.00000 -> 0.00000 1.00000 0.00000
- joint spine_3_rz: axis 1.00000 0.00000 0.00000 -> 0.00000 0.00000 1.00000
- joint spine_4_rx: axis 0.00000 1.00000 0.00000 -> 1.00000 0.00000 0.00000
- joint spine_4_ry: axis 0.00000 0.00000 1.00000 -> 0.00000 1.00000 0.00000
- joint spine_4_rz: axis 1.00000 0.00000 0.00000 -> 0.00000 0.00000 1.00000
